Commit message: [cmake] Use jrl-cmakemodules standards. Rewrite CMakeLists.txt [urdf] Change talos_small.urdf to use the smaller STL meshes.
* depends on urdfdom>=0.2.9. does not depend on Catkin
* remove package.xml
* add submodule cmake

NOTE: ASSIMP is angry with the header of the bigger STL files like arm_1.stl

File: robots/talos_small.urdf (robot description, URDF)
Before this commit: robot talos, 44 links, 43 joints
Links:
- link arm_left_1_link: geometry collision mesh filename=package://talos_description/meshes/arm/arm_1_collision.STL scale=1 1 1; visual mesh filename=package://talos_description/meshes/arm/arm_1_collision.STL scale=1 1 1
- link arm_left_2_link: geometry collision mesh filename=package://talos_description/meshes/arm/arm_2_collision.STL scale=1 1 1; visual mesh filename=package://talos_description/meshes/arm/arm_2_collision.STL scale=1 1 1
- link arm_left_3_link: geometry collision mesh filename=package://talos_description/meshes/arm/arm_3_collision.STL scale=1 1 1; visual mesh filename=package://talos_description/meshes/arm/arm_3_collision.STL scale=1 1 1
- link arm_left_4_link: geometry collision mesh filename=package://talos_description/meshes/arm/arm_4_collision.STL scale=1 1 1; visual mesh filename=package://talos_description/meshes/arm/arm_4_collision.STL scale=1 1 1
- link arm_left_5_link: geometry collision mesh filename=package://talos_description/meshes/arm/arm_5_collision.STL scale=1 1 1; visual mesh filename=package://talos_description/meshes/arm/arm_5_collision.STL scale=1 1 1
- link arm_left_6_link: geometry collision mesh filename=package://talos_description/meshes/arm/arm_6_collision.STL scale=1 1 1; visual mesh filename=package://talos_description/meshes/arm/arm_6_collision.STL scale=1 1 1
- link arm_right_1_link: geometry collision mesh filename=package://talos_description/meshes/arm/arm_1_collision.STL scale=1 -1 1; visual mesh filename=package://talos_description/meshes/arm/arm_1_collision.STL scale=1 -1 1
- link arm_right_2_link: geometry collision mesh filename=package://talos_description/meshes/arm/arm_2_collision.STL scale=1 -1 1; visual mesh filename=package://talos_description/meshes/arm/arm_2_collision.STL scale=1 -1 1
- link arm_right_3_link: geometry collision mesh filename=package://talos_description/meshes/arm/arm_3_collision.STL scale=1 -1 1; visual mesh filename=package://talos_description/meshes/arm/arm_3_collision.STL scale=1 -1 1
- link arm_right_4_link: geometry collision mesh filename=package://talos_description/meshes/arm/arm_4_collision.STL scale=1 -1 1; visual mesh filename=package://talos_description/meshes/arm/arm_4_collision.STL scale=1 -1 1
- link arm_right_5_link: geometry collision mesh filename=package://talos_description/meshes/arm/arm_5_collision.STL scale=1 -1 1; visual mesh filename=package://talos_description/meshes/arm/arm_5_collision.STL scale=1 -1 1
- link arm_right_6_link: geometry collision mesh filename=package://talos_description/meshes/arm/arm_6_collision.STL scale=1 -1 1; visual mesh filename=package://talos_description/meshes/arm/arm_6_collision.STL scale=1 -1 1
- link arm_right_7_link: geometry collision mesh filename=package://talos_description/meshes/arm/arm_7_collision.STL scale=1 -1 1; visual mesh filename=package://talos_description/meshes/arm/arm_7_collision.STL scale=1 -1 1
- link rgbd_link: geometry collision box size=0.04 0.185 0.03
