Commit message: [urdf] Create talos_reduced.urdf. remove talos_small.urdf
* Arms have 8 DOF instead of 7 (include last gripper joint)
* include the grippers as a fixed joint

File: robots/talos_reduced.urdf (robot description, URDF)
Before this commit: robot talos, 44 links, 43 joints
Links:
- added link gripper_left_base_link, mass 0.61585; collision mesh filename=package://talos_description/meshes/gripper/base_link_collis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 scale=1 1 1; visual mesh filename=package://talos_description/meshes/gripper/base_link.STL scale=1 1 1
- added link gripper_left_fingertip_1_link, mass 0.02630; collision mesh filename=package://talos_description/meshes/gripper/fingertip_collis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 scale=1 1 1; visual mesh filename=package://talos_description/meshes/gripper/fingertip.STL scale=1 1 1
- added link gripper_left_fingertip_2_link, mass 0.02630; collision mesh filename=package://talos_description/meshes/gripper/fingertip_collis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 scale=1 1 1; visual mesh filename=package://talos_description/meshes/gripper/fingertip.STL scale=1 1 1
- added link gripper_left_fingertip_3_link, mass 0.02630; collision mesh filename=package://talos_description/meshes/gripper/fingertip_collis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 scale=1 1 1; visual mesh filename=package://talos_description/meshes/gripper/fingertip.STL scale=1 1 1
- added link gripper_left_inner_double_link, mass 0.11922; collision mesh filename=package://talos_description/meshes/gripper/inner_double_col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 scale=1 1 1; visual mesh filename=package://talos_description/meshes/gripper/inner_double.STL scale=1 1 1
- added link gripper_left_inner_single_link, mass 0.05356; collision mesh filename=package://talos_description/meshes/gripper/inner_single_col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 scale=1 1 1; visual mesh filename=package://talos_description/meshes/gripper/inner_single.STL scale=1 1 1
- added link gripper_left_motor_double_link, mass 0.16889; collision mesh filename=package://talos_description/meshes/gripper/gripper_motor_do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 scale=1 1 1; visual mesh filename=package://talos_description/meshes/gripper/gripper_motor_do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 scale=1 1 1
- added link gripper_left_motor_single_link, mass 0.14765; collision mesh filename=package://talos_description/meshes/gripper/gripper_motor_si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 scale=1 1 1; visual mesh filename=package://talos_description/meshes/gripper/gripper_motor_si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 scale=1 1 1
- added link gripper_right_base_link, mass 0.61585; collision mesh filename=package://talos_description/meshes/gripper/base_link_collis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 scale=1 1 1; visual mesh filename=package://talos_description/meshes/gripper/base_link.STL scale=1 1 1
- added link gripper_right_fingertip_1_link, mass 0.02630; collision mesh filename=package://talos_description/meshes/gripper/fingertip_collis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 scale=1 1 1; visual mesh filename=package://talos_description/meshes/gripper/fingertip.STL scale=1 1 1
- added link gripper_right_fingertip_2_link, mass 0.02630; collision mesh filename=package://talos_description/meshes/gripper/fingertip_collis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 scale=1 1 1; visual mesh filename=package://talos_description/meshes/gripper/fingertip.STL scale=1 1 1
- added link gripper_right_fingertip_3_link, mass 0.02630; collision mesh filename=package://talos_description/meshes/gripper/fingertip_collis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 scale=1 1 1; visual mesh filename=package://talos_description/meshes/gripper/fingertip.STL scale=1 1 1
- added link gripper_right_inner_double_link, mass 0.11922; collision mesh filename=package://talos_description/meshes/gripper/inner_double_col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 scale=1 1 1; visual mesh filename=package://talos_description/meshes/gripper/inner_double.STL scale=1 1 1
- added link gripper_right_inner_single_link, mass 0.05356; collision mesh filename=package://talos_description/meshes/gripper/inner_single_col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 scale=1 1 1; visual mesh filename=package://talos_description/meshes/gripper/inner_single.STL scale=1 1 1
- added link gripper_right_motor_double_link, mass 0.16889; collision mesh filename=package://talos_description/meshes/gripper/gripper_motor_do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 scale=1 1 1; visual mesh filename=package://talos_description/meshes/gripper/gripper_motor_do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 scale=1 1 1
- added link gripper_right_motor_single_link, mass 0.14765; collision mesh filename=package://talos_description/meshes/gripper/gripper_motor_si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 scale=1 1 1; visual mesh filename=package://talos_description/meshes/gripper/gripper_motor_si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 scale=1 1 1
Joints:
- added joint gripper_left_base_link_joint: type fixed, parent wrist_left_ft_tool_link, child gripper_left_base_link, origin xyz=0.00000 0.00000 -0.02875 rpy=0.0 0.0 0.0, axis 0 0 0
- added joint gripper_left_fingertip_1_joint: type fixed, parent gripper_left_inner_double_link, child gripper_left_fingertip_1_link, origin xyz=0.03200 0.04589 -0.06553 rpy=0.0 0.0 0.0, axis 1 0 0, limit lower=0.0 upper=1.0471975512 effort=100.0 velocity=1.0, mimic joint=gripper_left_joint multiplier=-1.0 offset=0.0
- added joint gripper_left_fingertip_2_joint: type fixed, parent gripper_left_inner_double_link, child gripper_left_fingertip_2_link, origin xyz=-0.03200 0.04589 -0.06553 rpy=0.0 0.0 0.0, axis 1 0 0, limit lower=0.0 upper=1.0471975512 effort=100.0 velocity=1.0, mimic joint=gripper_left_joint multiplier=-1.0 offset=0.0
- added joint gripper_left_fingertip_3_joint: type fixed, parent gripper_left_inner_single_link, child gripper_left_fingertip_3_link, origin xyz=0.00000 -0.04589 -0.06553 rpy=0.0 0.0 3.14159265359, axis 1 0 0, limit lower=0.0 upper=1.0471975512 effort=100.0 velocity=1.0, mimic joint=gripper_left_joint multiplier=-1.0 offset=0.0
- added joint gripper_left_inner_double_joint: type fixed, parent gripper_left_base_link, child gripper_left_inner_double_link, origin xyz=0.00000 0.00525 -0.05598 rpy=0.0 0.0 0.0, axis 1 0 0, limit lower=-1.0471975512 upper=0.0 effort=100.0 velocity=1.0, mimic joint=gripper_left_joint multiplier=1.0 offset=0.0
- added joint gripper_left_inner_single_joint: type fixed, parent gripper_left_base_link, child gripper_left_inner_single_link, origin xyz=0.00000 -0.00525 -0.05598 rpy=0.0 0.0 0.0, axis 1 0 0, limit lower=0.0 upper=1.0471975512 effort=100.0 velocity=1.0, mimic joint=gripper_left_joint multiplier=-1.0 offset=0.0
- added joint gripper_left_joint: type revolute, parent gripper_left_base_link, child gripper_left_motor_double_link, origin xyz=0.0 0.02025 -0.03 rpy=0.0 0.0 0.0, axis 1 0 0, limit lower=-1.0471975512 upper=0.0 effort=1.0 velocity=1.0
- added joint gripper_left_motor_single_joint: type fixed, parent gripper_left_base_link, child gripper_left_motor_single_link, origin xyz=0.00000 -0.02025 -0.03000 rpy=0.0 0.0 0.0, axis 1 0 0, limit lower=0.0 upper=1.0471975512 effort=100.0 velocity=1.0, mimic joint=gripper_left_joint multiplier=-1.0 offset=0.0
- added joint gripper_right_base_link_joint: type fixed, parent wrist_right_ft_tool_link, child gripper_right_base_link, origin xyz=0.00000 0.00000 -0.02875 rpy=0.0 0.0 0.0, axis 0 0 0
- added joint gripper_right_fingertip_1_joint: type fixed, parent gripper_right_inner_double_link, child gripper_right_fingertip_1_link, origin xyz=0.03200 0.04589 -0.06553 rpy=0.0 0.0 0.0, axis 1 0 0, limit lower=0.0 upper=1.0471975512 effort=100.0 velocity=1.0, mimic joint=gripper_right_joint multiplier=-1.0 offset=0.0
- added joint gripper_right_fingertip_2_joint: type fixed, parent gripper_right_inner_double_link, child gripper_right_fingertip_2_link, origin xyz=-0.03200 0.04589 -0.06553 rpy=0.0 0.0 0.0, axis 1 0 0, limit lower=0.0 upper=1.0471975512 effort=100.0 velocity=1.0, mimic joint=gripper_right_joint multiplier=-1.0 offset=0.0
- added joint gripper_right_fingertip_3_joint: type fixed, parent gripper_right_inner_single_link, child gripper_right_fingertip_3_link, origin xyz=0.00000 -0.04589 -0.06553 rpy=0.0 0.0 3.14159265359, axis 1 0 0, limit lower=0.0 upper=1.0471975512 effort=100.0 velocity=1.0, mimic joint=gripper_right_joint multiplier=-1.0 offset=0.0
- added joint gripper_right_inner_double_joint: type fixed, parent gripper_right_base_link, child gripper_right_inner_double_link, origin xyz=0.00000 0.00525 -0.05598 rpy=0.0 0.0 0.0, axis 1 0 0, limit lower=-1.0471975512 upper=0.0 effort=100.0 velocity=1.0, mimic joint=gripper_right_joint multiplier=1.0 offset=0.0
- added joint gripper_right_inner_single_joint: type fixed, parent gripper_right_base_link, child gripper_right_inner_single_link, origin xyz=0.00000 -0.00525 -0.05598 rpy=0.0 0.0 0.0, axis 1 0 0, limit lower=0.0 upper=1.0471975512 effort=100.0 velocity=1.0, mimic joint=gripper_right_joint multiplier=-1.0 offset=0.0
- added joint gripper_right_joint: type revolute, parent gripper_right_base_link, child gripper_right_motor_double_link, origin xyz=0.0 0.02025 -0.03 rpy=0.0 0.0 0.0, axis 1 0 0, limit lower=-1.0471975512 upper=0.0 effort=1.0 velocity=1.0
- added joint gripper_right_motor_single_joint: type fixed, parent gripper_right_base_link, child gripper_right_motor_single_link, origin xyz=0.00000 -0.02025 -0.03000 rpy=0.0 0.0 0.0, axis 1 0 0, limit lower=0.0 upper=1.0471975512 effort=100.0 velocity=1.0, mimic joint=gripper_right_joint multiplier=-1.0 offset=0.0
