Commit message: Update to the same model than the robot.

File: robots/talos_full_v2.urdf (robot description, URDF)
Before this commit: robot talos, 60 links, 59 joints
Links:
- link arm_left_1_link: mass 1.42896 -> 2.714567; geometry collision mesh filename=package://talos_description/meshes/arm/arm_1_collision.STL scale=1 1 1; visual mesh filename=package://talos_description/meshes/arm/arm_1.STL scale=1 1 1
- link arm_left_2_link: mass 1.67729 -> 2.425086; geometry collision mesh filename=package://talos_description/meshes/arm/arm_2_collision.STL scale=1 1 1; visual mesh filename=package://talos_description/meshes/arm/arm_2.STL scale=1 1 1
- link arm_left_3_link: mass 1.47029 -> 2.208741; geometry collision mesh filename=package://talos_description/meshes/arm/arm_3_collision.STL scale=1 1 1; visual mesh filename=package://talos_description/meshes/arm/arm_3.STL scale=1 1 1
- link arm_left_4_link: mass 1.10216 -> 0.877346; geometry collision mesh filename=package://talos_description/meshes/arm/arm_4_collision.STL scale=1 1 1; visual mesh filename=package://talos_description/meshes/arm/arm_4.STL scale=1 1 1
- link arm_left_5_link: mass 1.77792 -> 1.877923; geometry collision mesh filename=package://talos_description/meshes/arm/arm_5_collision.STL scale=1 1 1; visual mesh filename=package://talos_description/meshes/arm/arm_5.STL scale=1 1 1
- link arm_left_6_link: mass 0.30931 -> 0.40931; geometry collision mesh filename=package://talos_description/meshes/arm/arm_6_collision.STL scale=1 1 1; visual mesh filename=package://talos_description/meshes/arm/arm_6.STL scale=1 1 1
- link arm_left_7_link: geometry collision mesh filename=package://talos_description/meshes/arm/arm_7_collision.STL scale=1 1 1; visual mesh filename=package://talos_description/meshes/arm/arm_7.STL scale=1 1 1
- link arm_right_1_link: mass 1.42896 -> 2.714567; geometry collision mesh filename=package://talos_description/meshes/arm/arm_1_collision.STL scale=1 -1 1; visual mesh filename=package://talos_description/meshes/arm/arm_1.STL scale=1 -1 1
- link arm_right_2_link: mass 1.67729 -> 2.425086; geometry collision mesh filename=package://talos_description/meshes/arm/arm_2_collision.STL scale=1 -1 1; visual mesh filename=package://talos_description/meshes/arm/arm_2.STL scale=1 -1 1
- link arm_right_3_link: mass 1.47029 -> 2.208741; geometry collision mesh filename=package://talos_description/meshes/arm/arm_3_collision.STL scale=1 -1 1; visual mesh filename=package://talos_description/meshes/arm/arm_3.STL scale=1 -1 1
- link arm_right_4_link: mass 1.10216 -> 0.877346; geometry collision mesh filename=package://talos_description/meshes/arm/arm_4_collision.STL scale=1 -1 1; visual mesh filename=package://talos_description/meshes/arm/arm_4.STL scale=1 -1 1
- link arm_right_5_link: mass 1.77792 -> 1.877923; geometry collision mesh filename=package://talos_description/meshes/arm/arm_5_collision.STL scale=1 -1 1; visual mesh filename=package://talos_description/meshes/arm/arm_5.STL scale=1 -1 1
- link arm_right_6_link: mass 0.30931 -> 0.40931; geometry collision mesh filename=package://talos_description/meshes/arm/arm_6_collision.STL scale=1 -1 1; visual mesh filename=package://talos_description/meshes/arm/arm_6.STL scale=1 -1 1
- link arm_right_7_link: geometry collision mesh filename=package://talos_description/meshes/arm/arm_7_collision.STL scale=1 -1 1; visual mesh filename=package://talos_description/meshes/arm/arm_7.STL scale=1 -1 1
- link base_link: mass 13.53810 -> 15.36284; geometry collision mesh filename=package://talos_description/meshes/torso/base_link_collisio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 scale=1 1 1; visual mesh filename=package://talos_description/meshes/torso/base_link.STL scale=1 1 1
- link gripper_left_base_link: mass 0.61585 -> 0.637534; geometry collision mesh filename=package://talos_description/meshes/gripper/base_link_collis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 scale=1 1 1; visual mesh filename=package://talos_description/meshes/gripper/base_link.STL scale=1 1 1
- link gripper_left_fingertip_1_link: mass 0.02630 -> 0.026301; geometry collision mesh filename=package://talos_description/meshes/gripper/fingertip_collis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 scale=1 1 1; visual mesh filename=package://talos_description/meshes/gripper/fingertip.STL scale=1 1 1
- link gripper_left_fingertip_2_link: mass 0.02630 -> 0.026301; geometry collision mesh filename=package://talos_description/meshes/gripper/fingertip_collis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 scale=1 1 1; visual mesh filename=package://talos_description/meshes/gripper/fingertip.STL scale=1 1 1
- link gripper_left_fingertip_3_link: mass 0.02630 -> 0.026301; geometry collision mesh filename=package://talos_description/meshes/gripper/fingertip_collis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 scale=1 1 1; visual mesh filename=package://talos_description/meshes/gripper/fingertip.STL scale=1 1 1
- link gripper_left_inner_double_link: mass 0.11922 -> 0.087986; geometry collision mesh filename=package://talos_description/meshes/gripper/inner_double_col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 scale=1 1 1; visual mesh filename=package://talos_description/meshes/gripper/inner_double.STL scale=1 1 1
- link gripper_left_inner_single_link: mass 0.05356 -> 0.047177; geometry collision mesh filename=package://talos_description/meshes/gripper/inner_single_col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 scale=1 1 1; visual mesh filename=package://talos_description/meshes/gripper/inner_single.STL scale=1 1 1
- link gripper_left_motor_double_link: mass 0.16889 -> 0.134356; geometry collision mesh filename=package://talos_description/meshes/gripper/gripper_motor_do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 scale=1 1 1; visual mesh filename=package://talos_description/meshes/gripper/gripper_motor_do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 scale=1 1 1
- link gripper_left_motor_single_link: mass 0.14765 -> 0.107923; geometry collision mesh filename=package://talos_description/meshes/gripper/gripper_motor_si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 scale=1 1 1; visual mesh filename=package://talos_description/meshes/gripper/gripper_motor_si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 scale=1 1 1
- link gripper_right_base_link: mass 0.61585 -> 0.637534; geometry collision mesh filename=package://talos_description/meshes/gripper/base_link_collis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 scale=1 1 1; visual mesh filename=package://talos_description/meshes/gripper/base_link.STL scale=1 1 1
- link gripper_right_fingertip_1_link: mass 0.02630 -> 0.026301; geometry collision mesh filename=package://talos_description/meshes/gripper/fingertip_collis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 scale=1 1 1; visual mesh filename=package://talos_description/meshes/gripper/fingertip.STL scale=1 1 1
- link gripper_right_fingertip_2_link: mass 0.02630 -> 0.026301; geometry collision mesh filename=package://talos_description/meshes/gripper/fingertip_collis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 scale=1 1 1; visual mesh filename=package://talos_description/meshes/gripper/fingertip.STL scale=1 1 1
- link gripper_right_fingertip_3_link: mass 0.02630 -> 0.026301; geometry collision mesh filename=package://talos_description/meshes/gripper/fingertip_collis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 scale=1 1 1; visual mesh filename=package://talos_description/meshes/gripper/fingertip.STL scale=1 1 1
- link gripper_right_inner_double_link: mass 0.11922 -> 0.087986; geometry collision mesh filename=package://talos_description/meshes/gripper/inner_double_col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 scale=1 1 1; visual mesh filename=package://talos_description/meshes/gripper/inner_double.STL scale=1 1 1
- link gripper_right_inner_single_link: mass 0.05356 -> 0.047177; geometry collision mesh filename=package://talos_description/meshes/gripper/inner_single_col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 scale=1 1 1; visual mesh filename=package://talos_description/meshes/gripper/inner_single.STL scale=1 1 1
- link gripper_right_motor_double_link: mass 0.16889 -> 0.134356; geometry collision mesh filename=package://talos_description/meshes/gripper/gripper_motor_do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 scale=1 1 1; visual mesh filename=package://talos_description/meshes/gripper/gripper_motor_do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 scale=1 1 1
- link gripper_right_motor_single_link: mass 0.14765 -> 0.107923; geometry collision mesh filename=package://talos_description/meshes/gripper/gripper_motor_si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 scale=1 1 1; visual mesh filename=package://talos_description/meshes/gripper/gripper_motor_si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 scale=1 1 1
- link head_1_link: mass 0.65988 -> 0.73746; geometry collision mesh filename=package://talos_description/meshes/head/head_1_collision.stl scale=1 1 1; visual mesh filename=package://talos_description/meshes/head/head_1.stl scale=1 1 1
- link head_2_link: mass 1.40353 -> 1.443954; geometry collision mesh filename=package://talos_description/meshes/head/head_2_collision.stl scale=1 1 1; visual mesh filename=package://talos_description/meshes/head/head_2.stl scale=1 1 1
- link leg_left_1_link: mass 1.88569 -> 1.845591; geometry collision mesh filename=package://talos_description/meshes/v2/hip_z_collision.stl scale=1 1 1; visual mesh filename=package://talos_description/meshes/v2/hip_z_lo_res.stl scale=1 1 1
- link leg_left_2_link: mass 2.37607 -> 1.490952; geometry collision mesh filename=package://talos_description/meshes/v2/hip_x_collision.stl scale=1 1 1; visual mesh filename=package://talos_description/meshes/v2/hip_x_lo_res.stl scale=1 1 1
- link leg_left_3_link: mass 6.82734 -> 6.239871; geometry collision mesh filename=package://talos_description/meshes/v2/hip_y_collision.stl scale=1 1 1; visual mesh filename=package://talos_description/meshes/v2/hip_y_lo_res.stl scale=1 1 1
- link leg_left_4_link: mass 3.63668 -> 3.759951; geometry collision mesh filename=package://talos_description/meshes/v2/knee_collision.stl scale=1 1 1; visual mesh filename=package://talos_description/meshes/v2/knee_lo_res.stl scale=1 1 1
- link leg_left_5_link: mass 1.24433 -> 1.29096; geometry collision mesh filename=package://talos_description/meshes/v2/ankle_Y_collision.stl scale=1 1 1; visual mesh filename=package://talos_description/meshes/v2/ankle_Y_lo_res.stl scale=1 1 1
- link leg_left_6_link: mass 1.59457 -> 1.597773; geometry collision box size=0.21 0.13 0.02; visual mesh filename=package://talos_description/meshes/v2/ankle_X_lo_res.stl scale=1 1 1
- link leg_right_1_link: mass 1.88569 -> 1.845591; geometry collision mesh filename=package://talos_description/meshes/v2/hip_z_collision.stl scale=1 -1 1; visual mesh filename=package://talos_description/meshes/v2/hip_z_lo_res.stl scale=1 -1 1
- link leg_right_2_link: mass 2.37607 -> 1.490952; geometry collision mesh filename=package://talos_description/meshes/v2/hip_x_collision.stl scale=1 -1 1; visual mesh filename=package://talos_description/meshes/v2/hip_x_lo_res.stl scale=1 -1 1
- link leg_right_3_link: mass 6.82734 -> 6.239871; geometry collision mesh filename=package://talos_description/meshes/v2/hip_y_collision.stl scale=1 -1 1; visual mesh filename=package://talos_description/meshes/v2/hip_y_lo_res.stl scale=1 -1 1
- link leg_right_4_link: mass 3.63668 -> 3.759951; geometry collision mesh filename=package://talos_description/meshes/v2/knee_collision.stl scale=1 -1 1; visual mesh filename=package://talos_description/meshes/v2/knee_lo_res.stl scale=1 -1 1
- link leg_right_5_link: mass 1.24433 -> 1.29096; geometry collision mesh filename=package://talos_description/meshes/v2/ankle_Y_collision.stl scale=1 -1 1; visual mesh filename=package://talos_description/meshes/v2/ankle_Y_lo_res.stl scale=1 -1 1
- link leg_right_6_link: mass 1.59457 -> 1.597773; geometry collision box size=0.21 0.13 0.02; visual mesh filename=package://talos_description/meshes/v2/ankle_X_lo_res.stl scale=1 -1 1
- link rgbd_link: geometry collision box size=0.04 0.185 0.03; visual mesh filename=package://talos_description/meshes/sensors/orbbec/orbbec.STL
- link torso_1_link: mass 3.02433 -> 2.294658; geometry collision mesh filename=package://talos_description/meshes/torso/torso_1.STL scale=1 1 1; visual mesh filename=package://talos_description/meshes/torso/torso_1.STL scale=1 1 1
- link torso_2_link: mass 17.55011 -> 16.97403; geometry collision mesh filename=package://talos_description/meshes/torso/torso_2_collision.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 scale=1 1 1; visual mesh filename=package://talos_description/meshes/torso/torso_2.STL scale=1 1 1
- link wrist_left_ft_link: mass 0.1 -> 0.095
- link wrist_left_ft_tool_link: mass 0.1 -> 0.001
- link wrist_right_ft_link: mass 0.1 -> 0.095
- link wrist_right_ft_tool_link: mass 0.1 -> 0.001
Joints:
- joint arm_left_1_joint: limit lower=-1.57079632679 upper=0.523598775598 effort=44.64 velocity=2.7 -> lower=-1.57079632679 upper=0.785398163397 effort=100.0 velocity=2.7
- joint arm_left_2_joint: limit lower=0.0 upper=2.87979326579 effort=22.32 velocity=3.66 -> lower=0.00872664625997 upper=2.87106661953 effort=100.0 velocity=3.66
- joint arm_left_3_joint: limit lower=-2.44346095279 upper=2.44346095279 effort=17.86 velocity=4.58 -> lower=-2.42600766027 upper=2.42600766027 effort=70.0 velocity=4.58
- joint arm_left_4_joint: limit lower=-2.35619449019 upper=0.0 effort=17.86 velocity=4.58 -> lower=-2.23402144255 upper=0.00349065850399 effort=70.0 velocity=4.58
- joint arm_left_5_joint: limit lower=-2.53072741539 upper=2.53072741539 effort=3 velocity=1.95 -> lower=-2.51327412287 upper=2.51327412287 effort=20.0 velocity=1.95
- joint arm_left_6_joint: limit lower=-1.3962634016 upper=1.3962634016 effort=6.6 velocity=1.76 -> lower=-1.37008346282 upper=1.37008346282 effort=8.0 velocity=1.76
- joint arm_left_7_joint: limit lower=-0.698131700798 upper=0.698131700798 effort=6.6 velocity=1.76 -> lower=-0.680678408278 upper=0.680678408278 effort=8.0 velocity=1.76
- joint arm_right_1_joint: limit lower=-0.523598775598 upper=1.57079632679 effort=44.64 velocity=2.7 -> lower=-0.785398163397 upper=1.57079632679 effort=100.0 velocity=2.7
- joint arm_right_2_joint: limit lower=-2.87979326579 upper=0.0 effort=22.32 velocity=3.66 -> lower=-2.87106661953 upper=-0.00872664625997 effort=100.0 velocity=3.66
- joint arm_right_3_joint: limit lower=-2.44346095279 upper=2.44346095279 effort=17.86 velocity=4.58 -> lower=-2.42600766027 upper=2.42600766027 effort=70.0 velocity=4.58
- joint arm_right_4_joint: limit lower=-2.35619449019 upper=0.0 effort=17.86 velocity=4.58 -> lower=-2.23402144255 upper=0.00349065850399 effort=70.0 velocity=4.58
- joint arm_right_5_joint: limit lower=-2.53072741539 upper=2.53072741539 effort=3 velocity=1.95 -> lower=-2.51327412287 upper=2.51327412287 effort=20.0 velocity=1.95
- joint arm_right_6_joint: limit lower=-1.3962634016 upper=1.3962634016 effort=6.6 velocity=1.76 -> lower=-1.37008346282 upper=1.37008346282 effort=8.0 velocity=1.76
- joint arm_right_7_joint: limit lower=-0.698131700798 upper=0.698131700798 effort=6.6 velocity=1.76 -> lower=-0.680678408278 upper=0.680678408278 effort=8.0 velocity=1.76
- joint gripper_left_joint: limit lower=-1.0471975512 upper=0.0 effort=1.0 velocity=1.0 -> lower=-0.959931088597 upper=0.0 effort=1.0 velocity=1.0
- joint gripper_right_joint: limit lower=-1.0471975512 upper=0.0 effort=1.0 velocity=1.0 -> lower=-0.959931088597 upper=0.0 effort=1.0 velocity=1.0
- joint head_1_joint: limit lower=-0.261799387799 upper=0.785398163397 effort=8.0 velocity=1.0 -> lower=-0.209439510239 upper=0.785398163397 effort=8.0 velocity=1.0; origin xyz=0.00000 0.00000 0.31600 rpy=0.0 0.0 0.0 -> xyz=0.02000 0.00000 0.32100 rpy=0.0 0.0 0.0
- joint leg_left_5_joint: limit lower=-1.309 upper=0.768 effort=160 velocity=5.8 -> lower=-1.27 upper=0.68 effort=160 velocity=5.8
- joint leg_right_5_joint: limit lower=-1.309 upper=0.768 effort=160 velocity=5.8 -> lower=-1.27 upper=0.68 effort=160 velocity=5.8
- joint rgbd_joint: origin xyz=0.066 0.0 0.1982 rpy=0 0 0 -> xyz=0.066 0.0 0.1982 rpy=0.0 0.0 0.0
- joint torso_1_joint: limit lower=-1.308996939 upper=1.308996939 effort=78.0 velocity=5.4 -> lower=-1.25663706144 upper=1.25663706144 effort=200.0 velocity=5.4
- joint torso_2_joint: limit lower=-0.261799387799 upper=0.785398163397 effort=78.0 velocity=5.4 -> lower=-0.226892802759 upper=0.733038285838 effort=200.0 velocity=5.4

File: urdf/arm/arm_v1.urdf.xacro (robot description, xacro)
@@ -9,7 +9,7 @@
 <robot xmlns:xacro="http://ros.org/wiki/xacro">
   <!--File includes-->
-  <xacro:include filename="$(find talos_data)/urdf/deg_to_rad.xacro" />
-  <xacro:include filename="$(find talos_data)/urdf/arm/wrist.urdf.xacro" />
-  <xacro:include filename="$(find talos_data)/urdf/arm/arm.transmission.xacro" />
+  <xacro:include filename="$(find talos_description)/urdf/deg_to_rad.xacro" />
+  <xacro:include filename="$(find talos_description)/urdf/arm/wrist.urdf.xacro" />
+  <xacro:include filename="$(find talos_description)/urdf/arm/arm.transmission.xacro" />
   <!--Constant parameters-->
   <xacro:property name="arm_friction"       value="1.0" />
@@ -19,8 +19,8 @@
   <xacro:property name="arm_3_max_vel"      value="4.58" />
   <xacro:property name="arm_4_max_vel"      value="4.58" />
-  <xacro:property name="arm_1_max_effort"   value="44.64" />
-  <xacro:property name="arm_2_max_effort"   value="22.32" />
-  <xacro:property name="arm_3_max_effort"   value="17.86" />
-  <xacro:property name="arm_4_max_effort"   value="17.86" />
+  <xacro:property name="arm_1_max_effort"   value="100.0" />
+  <xacro:property name="arm_2_max_effort"   value="100.0" />
+  <xacro:property name="arm_3_max_effort"   value="70.0" />
+  <xacro:property name="arm_4_max_effort"   value="70.0" />
   <xacro:property name="arm_eps"            value="0.02" />
   <xacro:macro name="talos_arm" params="name parent side reflect">
@@ -29,5 +29,4 @@
     <!--************************-->
     <link name="${name}_${side}_1_link">
-      <!-- TODO: Missing reflects of inertias -->
       <inertial>
         <origin xyz="-0.01346 ${reflect*0.09130} 0.04812" rpy="0.00000 0.00000 0.00000"/>
@@ -41,5 +40,5 @@
         <origin xyz="0 0 0" rpy="0 0 0" />
         <geometry>
-          <mesh filename="package://talos_data/meshes/arm/arm_1.STL" scale="1 ${reflect} 1"/>
+          <mesh filename="package://talos_description/meshes/arm/arm_1.STL" scale="1 ${reflect} 1"/>
         </geometry>
         <material name="DarkGrey" />
@@ -48,5 +47,5 @@
        <origin xyz="0 0 0" rpy="0 0 0" />
         <geometry>
-          <mesh filename="package://talos_data/meshes/arm/arm_1_collision.STL" scale="1 ${reflect} 1"/>
+          <mesh filename="package://talos_description/meshes/arm/arm_1_collision.STL" scale="1 ${reflect} 1"/>
         </geometry>
       </collision>
@@ -77,12 +76,12 @@
         <origin xyz="0 0 0" rpy="0 0 0" />
         <geometry>
-          <mesh filename="package://talos_data/meshes/arm/arm_2.STL" scale="1 ${reflect} 1"/>
-        </geometry>
-        <material name="DarkGrey" />
-      </visual>
-      <collision>
-        <origin xyz="0 0 0" rpy="0 0 0" />
-        <geometry>
-          <mesh filename="package://talos_data/meshes/arm/arm_2_collision.STL" scale="1 ${reflect} 1"/>
+          <mesh filename="package://talos_description/meshes/arm/arm_2.STL" scale="1 ${reflect} 1"/>
+        </geometry>
+        <material name="DarkGrey" />
+      </visual>
+      <collision>
+        <origin xyz="0 0 0" rpy="0 0 0" />
+        <geometry>
+          <mesh filename="package://talos_description/meshes/arm/arm_2_collision.STL" scale="1 ${reflect} 1"/>
         </geometry>
       </collision>
@@ -94,5 +93,5 @@
               rpy="${0.00000 * deg_to_rad} ${0.00000 * deg_to_rad} ${0.00000 * deg_to_rad}"/>
       <axis xyz="1 0 0" />
-      <limit lower="${(-82.50000 + 82.5*reflect)* deg_to_rad}" upper="${(82.50000 + 82.5000*reflect)* deg_to_rad}" effort="${arm_2_max_effort}" velocity="${arm_2_max_vel}" />
+      <limit lower="${(-82.0000 + 82.5000*reflect)* deg_to_rad}" upper="${(82.50000 + 82.0000*reflect)* deg_to_rad}" effort="${arm_2_max_effort}" velocity="${arm_2_max_vel}" />
       <dynamics friction="${arm_friction}" damping="${arm_damping}"/>
 <!--        <safety_controller k_position="20"
@@ -113,12 +112,12 @@
         <origin xyz="0 0 0" rpy="0 0 0" />
         <geometry>
-          <mesh filename="package://talos_data/meshes/arm/arm_3.STL" scale="1 ${reflect} 1"/>
-        </geometry>
-        <material name="DarkGrey" />
-      </visual>
-      <collision>
-        <origin xyz="0 0 0" rpy="0 0 0" />
-        <geometry>
-          <mesh filename="package://talos_data/meshes/arm/arm_3_collision.STL" scale="1 ${reflect} 1"/>
+          <mesh filename="package://talos_description/meshes/arm/arm_3.STL" scale="1 ${reflect} 1"/>
+        </geometry>
+        <material name="DarkGrey" />
+      </visual>
+      <collision>
+        <origin xyz="0 0 0" rpy="0 0 0" />
+        <geometry>
+          <mesh filename="package://talos_description/meshes/arm/arm_3_collision.STL" scale="1 ${reflect} 1"/>
         </geometry>
       </collision>
@@ -130,5 +129,5 @@
               rpy="${0.00000 * deg_to_rad} ${0.00000 * deg_to_rad} ${0.00000 * deg_to_rad}"/>
       <axis xyz="0 0 1" />
-      <limit lower="${-140.0 * deg_to_rad}" upper="${140.0 * deg_to_rad}" effort="${arm_3_max_effort}" velocity="${arm_3_max_vel}" />
+      <limit lower="${-139.0 * deg_to_rad}" upper="${139.0 * deg_to_rad}" effort="${arm_3_max_effort}" velocity="${arm_3_max_vel}" />
       <dynamics friction="${arm_friction}" damping="${arm_damping}"/>
 <!--       <safety_controller k_position="20"
@@ -152,12 +151,12 @@
         <origin xyz="0 0 0" rpy="0 0 0" />
         <geometry>
-          <mesh filename="package://talos_data/meshes/arm/arm_4.STL" scale="1 ${reflect} 1"/>
-        </geometry>
-        <material name="DarkGrey" />
-      </visual>
-      <collision>
-        <origin xyz="0 0 0" rpy="0 0 0" />
-        <geometry>
-          <mesh filename="package://talos_data/meshes/arm/arm_4_collision.STL" scale="1 ${reflect} 1"/>
+          <mesh filename="package://talos_description/meshes/arm/arm_4.STL" scale="1 ${reflect} 1"/>
+        </geometry>
+        <material name="DarkGrey" />
+      </visual>
+      <collision>
+        <origin xyz="0 0 0" rpy="0 0 0" />
+        <geometry>
+          <mesh filename="package://talos_description/meshes/arm/arm_4_collision.STL" scale="1 ${reflect} 1"/>
         </geometry>
       </collision>
@@ -169,5 +168,5 @@
               rpy="${0.00000 * deg_to_rad} ${0.00000 * deg_to_rad} ${0.00000 * deg_to_rad}"/>
       <axis xyz="0 1 0" />
-      <limit lower="${-135.0 * deg_to_rad}" upper="${0.0 * deg_to_rad}" effort="${arm_4_max_effort}" velocity="${arm_4_max_vel}" />
+      <limit lower="${-128.0 * deg_to_rad}" upper="${0.2 * deg_to_rad}" effort="${arm_4_max_effort}" velocity="${arm_4_max_vel}" />
       <dynamics friction="${arm_friction}" damping="${arm_damping}"/>
 <!--       <safety_controller k_position="20"
@@ -213,8 +212,5 @@
      <xacro:talos_wrist name="arm" parent="${name}_${side}_4_link" side="${side}" reflect="${reflect}" />
     <!-- extensions -->
-    <xacro:talos_arm_simple_transmission name="${name}" side="${side}" number="1" reduction="1.0" />
-    <xacro:talos_arm_simple_transmission name="${name}" side="${side}" number="2" reduction="1.0" />
-    <xacro:talos_arm_simple_transmission name="${name}" side="${side}" number="3" reduction="1.0" />
-    <xacro:talos_arm_simple_transmission name="${name}" side="${side}" number="4" reduction="1.0" />
+    <xacro:include filename="$(find talos_description)/urdf/arm/${side}_arm.transmissions.urdf.xacro" />
   </xacro:macro>
 </robot>
