Commit message: Introduces talos_gazebo with flexibilities.

File: robots/talos_full_v1.urdf.xacro (robot description, xacro)
@@ -12,14 +12,14 @@
         xmlns:interface="http://playerstage.sourceforge.net/gazebo/xmlschema/#interface">
   <xacro:if value="$(arg enable_crane)">
-    <xacro:include filename="$(find talos_description)/urdf/crane/crane.urdf.xacro" />
+    <xacro:include filename="$(find talos_data)/urdf/crane/crane.urdf.xacro" />
   </xacro:if>
-  <xacro:include filename="$(find talos_description)/urdf/torso/torso.urdf.xacro" />
-  <xacro:include filename="$(find talos_description)/urdf/head/head.urdf.xacro" />
+  <xacro:include filename="$(find talos_data)/urdf/torso/torso.urdf.xacro" />
+  <xacro:include filename="$(find talos_data)/urdf/head/head.urdf.xacro" />
   <!--arm_v1 loadded because of the different joint range for 1st DoF-->
-  <xacro:include filename="$(find talos_description)/urdf/arm/arm_v1.urdf.xacro" />
-  <xacro:include filename="$(find talos_description)/urdf/sensors/ftsensor.urdf.xacro" />
-  <xacro:include filename="$(find talos_description)/urdf/gripper/gripper.urdf.xacro" />
-  <xacro:include filename="$(find talos_description)/urdf/leg/leg.urdf.xacro" />
-  <xacro:include filename="$(find talos_description)/urdf/leg/foot_collision_$(arg foot_collision).urdf.xacro" />
+  <xacro:include filename="$(find talos_data)/urdf/arm/arm_v1.urdf.xacro" />
+  <xacro:include filename="$(find talos_data)/urdf/sensors/ftsensor.urdf.xacro" />
+  <xacro:include filename="$(find talos_data)/urdf/gripper/gripper.urdf.xacro" />
+  <xacro:include filename="$(find talos_data)/urdf/leg/leg.urdf.xacro" />
+  <xacro:include filename="$(find talos_data)/urdf/leg/foot_collision_$(arg foot_collision).urdf.xacro" />
   <xacro:include filename="$(find talos_description_inertial)/urdf/inertial.xacro" />
   <xacro:talos_torso name="torso" />
@@ -37,6 +37,6 @@
   <xacro:talos_leg prefix="right" reflect="-1" />
   <!-- Generic simulator_gazebo plugins -->
-  <xacro:include filename="$(find talos_description)/gazebo/gazebo.urdf.xacro" />
+  <xacro:include filename="$(find talos_data)/gazebo/gazebo.urdf.xacro" />
   <!-- Materials for visualization -->
-  <xacro:include filename="$(find talos_description)/urdf/materials.urdf.xacro" />
+  <xacro:include filename="$(find talos_data)/urdf/materials.urdf.xacro" />
 </robot>

File: robots/talos_full_v2.urdf.xacro (robot description, xacro)
@@ -12,14 +12,20 @@
         xmlns:interface="http://playerstage.sourceforge.net/gazebo/xmlschema/#interface">
   <xacro:if value="$(arg enable_crane)">
-    <xacro:include filename="$(find talos_description)/urdf/crane/crane.urdf.xacro" />
+    <xacro:include filename="$(find talos_data)/urdf/crane/crane.urdf.xacro" />
   </xacro:if>
-  <xacro:include filename="$(find talos_description)/urdf/torso/torso.urdf.xacro" />
-  <xacro:include filename="$(find talos_description)/urdf/head/head.urdf.xacro" />
+  <xacro:include filename="$(find talos_data)/urdf/torso/torso.urdf.xacro" />
+  <xacro:include filename="$(find talos_data)/urdf/head/head.urdf.xacro" />
   <!--arm_v1 loadded because of the different joint range for 1st DoF-->
-  <xacro:include filename="$(find talos_description)/urdf/arm/arm_v2.urdf.xacro" />
-  <xacro:include filename="$(find talos_description)/urdf/sensors/ftsensor.urdf.xacro" />
-  <xacro:include filename="$(find talos_description)/urdf/gripper/gripper.urdf.xacro" />
-  <xacro:include filename="$(find talos_description)/urdf/leg/leg.urdf.xacro" />
-  <xacro:include filename="$(find talos_description)/urdf/leg/foot_collision_$(arg foot_collision).urdf.xacro" />
+  <xacro:include filename="$(find talos_data)/urdf/arm/arm_v2.urdf.xacro" />
+  <xacro:include filename="$(find talos_data)/urdf/sensors/ftsensor.urdf.xacro" />
+  <xacro:include filename="$(find talos_data)/urdf/gripper/gripper.urdf.xacro" />
+  <xacro:if value="$(arg enable_leg_passive)">
+    <xacro:include filename="$(find talos_data)/urdf/leg/leg_passive.urdf.xacro" />
+  </xacro:if>
+  <xacro:property name="var_enable_leg_passive" value="$(arg enable_leg_passive)"/>
+  <xacro:if value="${var_enable_leg_passive != 'true'}">
+    <xacro:include filename="$(find talos_data)/urdf/leg/leg.urdf.xacro" />
+  </xacro:if>
+  <xacro:include filename="$(find talos_data)/urdf/leg/foot_collision_$(arg foot_collision).urdf.xacro" />
   <xacro:include filename="$(find talos_description_inertial)/urdf/inertial.xacro" />
   <xacro:talos_torso name="torso" />
@@ -37,6 +43,6 @@
   <xacro:talos_leg prefix="right" reflect="-1" />
   <!-- Generic simulator_gazebo plugins -->
-  <xacro:include filename="$(find talos_description)/gazebo/gazebo.urdf.xacro" />
+  <xacro:include filename="$(find talos_data)/gazebo/gazebo.urdf.xacro" />
   <!-- Materials for visualization -->
-  <xacro:include filename="$(find talos_description)/urdf/materials.urdf.xacro" />
+  <xacro:include filename="$(find talos_data)/urdf/materials.urdf.xacro" />
 </robot>

File: robots/talos_lower_body.urdf.xacro (robot description, xacro)
@@ -11,7 +11,7 @@
         xmlns:controller="http://playerstage.sourceforge.net/gazebo/xmlschema/#controller"
         xmlns:interface="http://playerstage.sourceforge.net/gazebo/xmlschema/#interface">
-  <xacro:include filename="$(find talos_description)/urdf/sensors/ftsensor.urdf.xacro" />
-  <xacro:include filename="$(find talos_description)/urdf/leg/leg.urdf.xacro" />
-  <xacro:include filename="$(find talos_description)/urdf/leg/foot_collision_$(arg foot_collision).urdf.xacro" />
+  <xacro:include filename="$(find talos_data)/urdf/sensors/ftsensor.urdf.xacro" />
+  <xacro:include filename="$(find talos_data)/urdf/leg/leg.urdf.xacro" />
+  <xacro:include filename="$(find talos_data)/urdf/leg/foot_collision_$(arg foot_collision).urdf.xacro" />
   <xacro:include filename="$(find talos_description_inertial)/urdf/inertial.xacro" />
     <!--************************-->
@@ -29,5 +29,5 @@
         <origin xyz="0 0 0" rpy="0 0 0" />
         <geometry>
-          <mesh filename="package://talos_description/meshes/torso/base_link.STL" scale="1 1 1"/>
+          <mesh filename="package://talos_data/meshes/torso/base_link.STL" scale="1 1 1"/>
         </geometry>
         <material name="LightGrey" />
@@ -36,5 +36,5 @@
         <origin xyz="0 0 0" rpy="0 0 0" />
         <geometry>
-          <mesh filename="package://talos_description/meshes/torso/base_link_collision.STL" scale="1 1 1"/>
+          <mesh filename="package://talos_data/meshes/torso/base_link_collision.STL" scale="1 1 1"/>
         </geometry>
       </collision>
@@ -43,6 +43,6 @@
   <xacro:talos_leg prefix="right" reflect="-1" />
   <!-- Generic simulator_gazebo plugins -->
-  <xacro:include filename="$(find talos_description)/gazebo/gazebo.urdf.xacro" />
+  <xacro:include filename="$(find talos_data)/gazebo/gazebo.urdf.xacro" />
   <!-- Materials for visualization -->
-  <xacro:include filename="$(find talos_description)/urdf/materials.urdf.xacro" />
+  <xacro:include filename="$(find talos_data)/urdf/materials.urdf.xacro" />
 </robot>

File: urdf/arm/arm_v1.urdf.xacro (robot description, xacro)
@@ -9,7 +9,7 @@
 <robot xmlns:xacro="http://ros.org/wiki/xacro">
   <!--File includes-->
-  <xacro:include filename="$(find talos_description)/urdf/deg_to_rad.xacro" />
-  <xacro:include filename="$(find talos_description)/urdf/arm/wrist.urdf.xacro" />
-  <xacro:include filename="$(find talos_description)/urdf/arm/arm.transmission.xacro" />
+  <xacro:include filename="$(find talos_data)/urdf/deg_to_rad.xacro" />
+  <xacro:include filename="$(find talos_data)/urdf/arm/wrist.urdf.xacro" />
+  <xacro:include filename="$(find talos_data)/urdf/arm/arm.transmission.xacro" />
   <!--Constant parameters-->
   <xacro:property name="arm_friction"       value="1.0" />
@@ -40,5 +40,5 @@
         <origin xyz="0 0 0" rpy="0 0 0" />
         <geometry>
-          <mesh filename="package://talos_description/meshes/arm/arm_1.STL" scale="1 ${reflect} 1"/>
+          <mesh filename="package://talos_data/meshes/arm/arm_1.STL" scale="1 ${reflect} 1"/>
         </geometry>
         <material name="DarkGrey" />
@@ -47,5 +47,5 @@
        <origin xyz="0 0 0" rpy="0 0 0" />
         <geometry>
-          <mesh filename="package://talos_description/meshes/arm/arm_1_collision.STL" scale="1 ${reflect} 1"/>
+          <mesh filename="package://talos_data/meshes/arm/arm_1_collision.STL" scale="1 ${reflect} 1"/>
         </geometry>
       </collision>
@@ -76,12 +76,12 @@
         <origin xyz="0 0 0" rpy="0 0 0" />
         <geometry>
-          <mesh filename="package://talos_description/meshes/arm/arm_2.STL" scale="1 ${reflect} 1"/>
-        </geometry>
-        <material name="DarkGrey" />
-      </visual>
-      <collision>
-        <origin xyz="0 0 0" rpy="0 0 0" />
-        <geometry>
-          <mesh filename="package://talos_description/meshes/arm/arm_2_collision.STL" scale="1 ${reflect} 1"/>
+          <mesh filename="package://talos_data/meshes/arm/arm_2.STL" scale="1 ${reflect} 1"/>
+        </geometry>
+        <material name="DarkGrey" />
+      </visual>
+      <collision>
+        <origin xyz="0 0 0" rpy="0 0 0" />
+        <geometry>
+          <mesh filename="package://talos_data/meshes/arm/arm_2_collision.STL" scale="1 ${reflect} 1"/>
         </geometry>
       </collision>
@@ -112,12 +112,12 @@
         <origin xyz="0 0 0" rpy="0 0 0" />
         <geometry>
-          <mesh filename="package://talos_description/meshes/arm/arm_3.STL" scale="1 ${reflect} 1"/>
-        </geometry>
-        <material name="DarkGrey" />
-      </visual>
-      <collision>
-        <origin xyz="0 0 0" rpy="0 0 0" />
-        <geometry>
-          <mesh filename="package://talos_description/meshes/arm/arm_3_collision.STL" scale="1 ${reflect} 1"/>
+          <mesh filename="package://talos_data/meshes/arm/arm_3.STL" scale="1 ${reflect} 1"/>
+        </geometry>
+        <material name="DarkGrey" />
+      </visual>
+      <collision>
+        <origin xyz="0 0 0" rpy="0 0 0" />
+        <geometry>
+          <mesh filename="package://talos_data/meshes/arm/arm_3_collision.STL" scale="1 ${reflect} 1"/>
         </geometry>
       </collision>
@@ -151,12 +151,12 @@
         <origin xyz="0 0 0" rpy="0 0 0" />
         <geometry>
-          <mesh filename="package://talos_description/meshes/arm/arm_4.STL" scale="1 ${reflect} 1"/>
-        </geometry>
-        <material name="DarkGrey" />
-      </visual>
-      <collision>
-        <origin xyz="0 0 0" rpy="0 0 0" />
-        <geometry>
-          <mesh filename="package://talos_description/meshes/arm/arm_4_collision.STL" scale="1 ${reflect} 1"/>
+          <mesh filename="package://talos_data/meshes/arm/arm_4.STL" scale="1 ${reflect} 1"/>
+        </geometry>
+        <material name="DarkGrey" />
+      </visual>
+      <collision>
+        <origin xyz="0 0 0" rpy="0 0 0" />
+        <geometry>
+          <mesh filename="package://talos_data/meshes/arm/arm_4_collision.STL" scale="1 ${reflect} 1"/>
         </geometry>
       </collision>
@@ -212,5 +212,5 @@
      <xacro:talos_wrist name="arm" parent="${name}_${side}_4_link" side="${side}" reflect="${reflect}" />
     <!-- extensions -->
-    <xacro:include filename="$(find talos_description)/urdf/arm/${side}_arm.transmissions.urdf.xacro" />
+    <xacro:include filename="$(find talos_data)/urdf/arm/${side}_arm.transmissions.urdf.xacro" />
   </xacro:macro>
 </robot>

File: urdf/arm/arm_v2.urdf.xacro (robot description, xacro)
@@ -9,7 +9,7 @@
 <robot xmlns:xacro="http://ros.org/wiki/xacro">
   <!--File includes-->
-  <xacro:include filename="$(find talos_description)/urdf/deg_to_rad.xacro" />
-  <xacro:include filename="$(find talos_description)/urdf/arm/wrist.urdf.xacro" />
-  <xacro:include filename="$(find talos_description)/urdf/arm/arm.transmission.xacro" />
+  <xacro:include filename="$(find talos_data)/urdf/deg_to_rad.xacro" />
+  <xacro:include filename="$(find talos_data)/urdf/arm/wrist.urdf.xacro" />
+  <xacro:include filename="$(find talos_data)/urdf/arm/arm.transmission.xacro" />
   <!--Constant parameters-->
   <xacro:property name="arm_friction"       value="1.0" />
@@ -33,5 +33,5 @@
         <origin xyz="0 0 0" rpy="0 0 0" />
         <geometry>
-          <mesh filename="package://talos_description/meshes/arm/arm_1.STL" scale="1 ${reflect} 1"/>
+          <mesh filename="package://talos_data/meshes/arm/arm_1.STL" scale="1 ${reflect} 1"/>
         </geometry>
         <material name="DarkGrey" />
@@ -40,5 +40,5 @@
        <origin xyz="0 0 0" rpy="0 0 0" />
         <geometry>
-          <mesh filename="package://talos_description/meshes/arm/arm_1_collision.STL" scale="1 ${reflect} 1"/>
+          <mesh filename="package://talos_data/meshes/arm/arm_1_collision.STL" scale="1 ${reflect} 1"/>
         </geometry>
       </collision>
@@ -64,5 +64,5 @@
         <origin xyz="0 0 0" rpy="0 0 0" />
         <geometry>
-          <mesh filename="package://talos_description/meshes/arm/arm_2.STL" scale="1 ${reflect} 1"/>
+          <mesh filename="package://talos_data/meshes/arm/arm_2.STL" scale="1 ${reflect} 1"/>
         </geometry>
         <material name="DarkGrey" />
@@ -71,5 +71,5 @@
         <origin xyz="0 0 0" rpy="0 0 0" />
         <geometry>
-          <mesh filename="package://talos_description/meshes/arm/arm_2_collision.STL" scale="1 ${reflect} 1"/>
+          <mesh filename="package://talos_data/meshes/arm/arm_2_collision.STL" scale="1 ${reflect} 1"/>
         </geometry>
       </collision>
@@ -93,5 +93,5 @@
         <origin xyz="0 0 0" rpy="0 0 0" />
         <geometry>
-          <mesh filename="package://talos_description/meshes/arm/arm_3.STL" scale="1 ${reflect} 1"/>
+          <mesh filename="package://talos_data/meshes/arm/arm_3.STL" scale="1 ${reflect} 1"/>
         </geometry>
         <material name="DarkGrey" />
@@ -100,5 +100,5 @@
         <origin xyz="0 0 0" rpy="0 0 0" />
         <geometry>
-          <mesh filename="package://talos_description/meshes/arm/arm_3_collision.STL" scale="1 ${reflect} 1"/>
+          <mesh filename="package://talos_data/meshes/arm/arm_3_collision.STL" scale="1 ${reflect} 1"/>
         </geometry>
       </collision>
@@ -125,5 +125,5 @@
         <origin xyz="0 0 0" rpy="0 0 0" />
         <geometry>
-          <mesh filename="package://talos_description/meshes/arm/arm_4.STL" scale="1 ${reflect} 1"/>
+          <mesh filename="package://talos_data/meshes/arm/arm_4.STL" scale="1 ${reflect} 1"/>
         </geometry>
         <material name="DarkGrey" />
@@ -132,5 +132,5 @@
         <origin xyz="0 0 0" rpy="0 0 0" />
         <geometry>
-          <mesh filename="package://talos_description/meshes/arm/arm_4_collision.STL" scale="1 ${reflect} 1"/>
+          <mesh filename="package://talos_data/meshes/arm/arm_4_collision.STL" scale="1 ${reflect} 1"/>
         </geometry>
       </collision>
@@ -186,5 +186,5 @@
      <xacro:talos_wrist name="arm" parent="${name}_${side}_4_link" side="${side}" reflect="${reflect}" />
     <!-- extensions -->
-    <xacro:include filename="$(find talos_description)/urdf/arm/${side}_arm.transmissions.urdf.xacro" />
+    <xacro:include filename="$(find talos_data)/urdf/arm/${side}_arm.transmissions.urdf.xacro" />
   </xacro:macro>
 </robot>

File: urdf/arm/left_arm.transmissions.urdf.xacro (robot description, xacro)
@@ -9,5 +9,5 @@
 <robot xmlns:xacro="http://ros.org/wiki/xacro">
   <!--File includes-->
-  <xacro:include filename="$(find talos_description)/urdf/arm/arm.transmission.xacro" />
+  <xacro:include filename="$(find talos_data)/urdf/arm/arm.transmission.xacro" />
   <xacro:include filename="$(find talos_description_calibration)/urdf/calibration/calibration_constants.urdf.xacro" />
   <!-- extensions -->

File: urdf/arm/left_wrist.transmissions.urdf.xacro (robot description, xacro)
@@ -9,5 +9,5 @@
 <robot xmlns:xacro="http://ros.org/wiki/xacro">
   <!--File includes-->
-  <xacro:include filename="$(find talos_description)/urdf/arm/wrist.transmission.xacro" />
+  <xacro:include filename="$(find talos_data)/urdf/arm/wrist.transmission.xacro" />
   <xacro:include filename="$(find talos_description_calibration)/urdf/calibration/calibration_constants.urdf.xacro" />
   <!-- extensions -->

File: urdf/arm/right_arm.transmissions.urdf.xacro (robot description, xacro)
@@ -9,5 +9,5 @@
 <robot xmlns:xacro="http://ros.org/wiki/xacro">
   <!--File includes-->
-  <xacro:include filename="$(find talos_description)/urdf/arm/arm.transmission.xacro" />
+  <xacro:include filename="$(find talos_data)/urdf/arm/arm.transmission.xacro" />
   <xacro:include filename="$(find talos_description_calibration)/urdf/calibration/calibration_constants.urdf.xacro" />
   <!-- extensions -->

File: urdf/arm/right_wrist.transmissions.urdf.xacro (robot description, xacro)
@@ -9,5 +9,5 @@
 <robot xmlns:xacro="http://ros.org/wiki/xacro">
   <!--File includes-->
-  <xacro:include filename="$(find talos_description)/urdf/arm/wrist.transmission.xacro" />
+  <xacro:include filename="$(find talos_data)/urdf/arm/wrist.transmission.xacro" />
   <xacro:include filename="$(find talos_description_calibration)/urdf/calibration/calibration_constants.urdf.xacro" />
   <!-- extensions -->

File: urdf/arm/wrist.urdf.xacro (robot description, xacro)
@@ -9,6 +9,6 @@
 <robot xmlns:xacro="http://ros.org/wiki/xacro">
   <!--File includes-->
-  <xacro:include filename="$(find talos_description)/urdf/deg_to_rad.xacro" />
-  <xacro:include filename="$(find talos_description)/urdf/arm/wrist.transmission.xacro" />
+  <xacro:include filename="$(find talos_data)/urdf/deg_to_rad.xacro" />
+  <xacro:include filename="$(find talos_data)/urdf/arm/wrist.transmission.xacro" />
   <!--Constant parameters-->
   <xacro:property name="wrist_friction"       value="1.0" />
@@ -30,5 +30,5 @@
         <origin xyz="0 0 0" rpy="0 0 0" />
         <geometry>
-          <mesh filename="package://talos_description/meshes/arm/arm_5.STL" scale="1 ${reflect} 1"/>
+          <mesh filename="package://talos_data/meshes/arm/arm_5.STL" scale="1 ${reflect} 1"/>
         </geometry>
         <material name="LightGrey" />
@@ -37,5 +37,5 @@
         <origin xyz="0 0 0" rpy="0 0 0" />
         <geometry>
-          <mesh filename="package://talos_description/meshes/arm/arm_5_collision.STL" scale="1 ${reflect} 1"/>
+          <mesh filename="package://talos_data/meshes/arm/arm_5_collision.STL" scale="1 ${reflect} 1"/>
         </geometry>
       </collision>
@@ -59,5 +59,5 @@
         <origin xyz="0 0 0" rpy="0 0 0" />
         <geometry>
-          <mesh filename="package://talos_description/meshes/arm/arm_6.STL" scale="1 ${reflect} 1"/>
+          <mesh filename="package://talos_data/meshes/arm/arm_6.STL" scale="1 ${reflect} 1"/>
         </geometry>
         <material name="LightGrey" />
@@ -66,5 +66,5 @@
         <origin xyz="0 0 0" rpy="0 0 0" />
         <geometry>
-          <mesh filename="package://talos_description/meshes/arm/arm_6_collision.STL" scale="1 ${reflect} 1"/>
+          <mesh filename="package://talos_data/meshes/arm/arm_6_collision.STL" scale="1 ${reflect} 1"/>
         </geometry>
       </collision>
@@ -88,5 +88,5 @@
         <origin xyz="0 0 0" rpy="0 0 0" />
         <geometry>
-          <mesh filename="package://talos_description/meshes/arm/arm_7.STL" scale="1 ${reflect} 1"/>
+          <mesh filename="package://talos_data/meshes/arm/arm_7.STL" scale="1 ${reflect} 1"/>
         </geometry>
         <material name="DarkGrey" />
@@ -95,5 +95,5 @@
         <origin xyz="0 0 0" rpy="0 0 0" />
         <geometry>
-          <mesh filename="package://talos_description/meshes/arm/arm_7_collision.STL" scale="1 ${reflect} 1"/>
+          <mesh filename="package://talos_data/meshes/arm/arm_7_collision.STL" scale="1 ${reflect} 1"/>
         </geometry>
       </collision>
@@ -136,5 +136,5 @@
     </gazebo>
     <!-- extensions -->
-    <xacro:include filename="$(find talos_description)/urdf/arm/${side}_wrist.transmissions.urdf.xacro" />
+    <xacro:include filename="$(find talos_data)/urdf/arm/${side}_wrist.transmissions.urdf.xacro" />
   </xacro:macro>
 </robot>

File: urdf/crane/crane.urdf.xacro (robot description, xacro)
@@ -9,5 +9,5 @@
 <robot xmlns:xacro="http://ros.org/wiki/xacro">
   <!--File includes-->
-  <xacro:include filename="$(find talos_description)/urdf/deg_to_rad.xacro" />
+  <xacro:include filename="$(find talos_data)/urdf/deg_to_rad.xacro" />
   <xacro:macro name="crane" params="parent">
     <link name="crane_link">
