Commit message: Introduces talos_gazebo with flexibilities.

File: urdf/gripper/gripper.urdf.xacro (robot description, xacro)
@@ -2,7 +2,7 @@
 <robot xmlns:xacro="http://ros.org/wiki/xacro">
   <!--File includes-->
-  <xacro:include filename="$(find talos_description)/urdf/deg_to_rad.xacro" />
-  <xacro:include filename="$(find talos_description)/urdf/gripper/gripper.transmission.xacro" />
-  <xacro:include filename="$(find talos_description)/urdf/gripper/gripper.gazebo.xacro" />
+  <xacro:include filename="$(find talos_data)/urdf/deg_to_rad.xacro" />
+  <xacro:include filename="$(find talos_data)/urdf/gripper/gripper.transmission.xacro" />
+  <xacro:include filename="$(find talos_data)/urdf/gripper/gripper.gazebo.xacro" />
   <xacro:macro name="talos_gripper" params="name parent reflect">
             <link name="${name}_base_link">
@@ -11,5 +11,5 @@
                 <origin xyz="0 0 0" rpy="0 0 0" />
                 <geometry>
-                  <mesh filename="package://talos_description/meshes/gripper/base_link.STL" scale="1 1 1"/>
+                  <mesh filename="package://talos_data/meshes/gripper/base_link.STL" scale="1 1 1"/>
                 </geometry>
                 <material name="DarkGrey"/>
@@ -18,5 +18,5 @@
                 <origin xyz="0 0 0" rpy="0 0 0" />
                 <geometry>
-                  <mesh filename="package://talos_description/meshes/gripper/base_link_collision.STL" scale="1 1 1"/>
+                  <mesh filename="package://talos_data/meshes/gripper/base_link_collision.STL" scale="1 1 1"/>
                 </geometry>
               </collision>
@@ -34,12 +34,12 @@
                 <origin xyz="0 0 0" rpy="0 0 0" />
                 <geometry>
-                  <mesh filename="package://talos_description/meshes/gripper/gripper_motor_double.STL" scale="1 1 1"/>
-                </geometry>
-              <material name="Orange"/>
-              </visual>
-              <collision>
-                <origin xyz="0 0 0" rpy="0 0 0" />
-                <geometry>
-                  <mesh filename="package://talos_description/meshes/gripper/gripper_motor_double_collision.STL" scale="1 1 1"/>
+                  <mesh filename="package://talos_data/meshes/gripper/gripper_motor_double.STL" scale="1 1 1"/>
+                </geometry>
+              <material name="Orange"/>
+              </visual>
+              <collision>
+                <origin xyz="0 0 0" rpy="0 0 0" />
+                <geometry>
+                  <mesh filename="package://talos_data/meshes/gripper/gripper_motor_double_collision.STL" scale="1 1 1"/>
                 </geometry>
               </collision>
@@ -59,12 +59,12 @@
                 <origin xyz="0 0 0" rpy="0 0 0" />
                 <geometry>
-                  <mesh filename="package://talos_description/meshes/gripper/inner_double.STL" scale="1 1 1"/>
-                </geometry>
-              <material name="Orange"/>
-              </visual>
-              <collision>
-                <origin xyz="0 0 0" rpy="0 0 0" />
-                <geometry>
-                  <mesh filename="package://talos_description/meshes/gripper/inner_double_collision.STL" scale="1 1 1"/>
+                  <mesh filename="package://talos_data/meshes/gripper/inner_double.STL" scale="1 1 1"/>
+                </geometry>
+              <material name="Orange"/>
+              </visual>
+              <collision>
+                <origin xyz="0 0 0" rpy="0 0 0" />
+                <geometry>
+                  <mesh filename="package://talos_data/meshes/gripper/inner_double_collision.STL" scale="1 1 1"/>
                 </geometry>
               </collision>
@@ -84,5 +84,5 @@
                 <origin xyz="0 0 0" rpy="0 0 0" />
                 <geometry>
-                  <mesh filename="package://talos_description/meshes/gripper/fingertip.STL" scale="1 1 1"/>
+                  <mesh filename="package://talos_data/meshes/gripper/fingertip.STL" scale="1 1 1"/>
                 </geometry>
               <material name="DarkGrey"/>
@@ -91,5 +91,5 @@
                 <origin xyz="0 0 0" rpy="0 0 0" />
                 <geometry>
-                  <mesh filename="package://talos_description/meshes/gripper/fingertip_collision.STL" scale="1 1 1"/>
+                  <mesh filename="package://talos_data/meshes/gripper/fingertip_collision.STL" scale="1 1 1"/>
                 </geometry>
               </collision>
@@ -109,5 +109,5 @@
                 <origin xyz="0 0 0" rpy="0 0 0" />
                 <geometry>
-                  <mesh filename="package://talos_description/meshes/gripper/fingertip.STL" scale="1 1 1"/>
+                  <mesh filename="package://talos_data/meshes/gripper/fingertip.STL" scale="1 1 1"/>
                 </geometry>
                 <material name="DarkGrey"/>
@@ -116,5 +116,5 @@
                 <origin xyz="0 0 0" rpy="0 0 0" />
                 <geometry>
-                  <mesh filename="package://talos_description/meshes/gripper/fingertip_collision.STL" scale="1 1 1"/>
+                  <mesh filename="package://talos_data/meshes/gripper/fingertip_collision.STL" scale="1 1 1"/>
                 </geometry>
               </collision>
@@ -134,12 +134,12 @@
                 <origin xyz="0 0 0" rpy="0 0 0" />
                 <geometry>
-                  <mesh filename="package://talos_description/meshes/gripper/gripper_motor_single.STL" scale="1 1 1"/>
-                </geometry>
-              <material name="Orange"/>
-              </visual>
-              <collision>
-                <origin xyz="0 0 0" rpy="0 0 0" />
-                <geometry>
-                  <mesh filename="package://talos_description/meshes/gripper/gripper_motor_single_collision.STL" scale="1 1 1"/>
+                  <mesh filename="package://talos_data/meshes/gripper/gripper_motor_single.STL" scale="1 1 1"/>
+                </geometry>
+              <material name="Orange"/>
+              </visual>
+              <collision>
+                <origin xyz="0 0 0" rpy="0 0 0" />
+                <geometry>
+                  <mesh filename="package://talos_data/meshes/gripper/gripper_motor_single_collision.STL" scale="1 1 1"/>
                 </geometry>
               </collision>
@@ -159,12 +159,12 @@
                 <origin xyz="0 0 0" rpy="0 0 0" />
                 <geometry>
-                  <mesh filename="package://talos_description/meshes/gripper/inner_single.STL" scale="1 1 1"/>
-                </geometry>
-              <material name="Orange"/>
-              </visual>
-              <collision>
-                <origin xyz="0 0 0" rpy="0 0 0" />
-                <geometry>
-                  <mesh filename="package://talos_description/meshes/gripper/inner_single_collision.STL" scale="1 1 1"/>
+                  <mesh filename="package://talos_data/meshes/gripper/inner_single.STL" scale="1 1 1"/>
+                </geometry>
+              <material name="Orange"/>
+              </visual>
+              <collision>
+                <origin xyz="0 0 0" rpy="0 0 0" />
+                <geometry>
+                  <mesh filename="package://talos_data/meshes/gripper/inner_single_collision.STL" scale="1 1 1"/>
                 </geometry>
               </collision>
@@ -184,5 +184,5 @@
                 <origin xyz="0 0 0" rpy="0 0 0" />
                 <geometry>
-                  <mesh filename="package://talos_description/meshes/gripper/fingertip.STL" scale="1 1 1"/>
+                  <mesh filename="package://talos_data/meshes/gripper/fingertip.STL" scale="1 1 1"/>
                 </geometry>
               <material name="DarkGrey"/>
@@ -191,5 +191,5 @@
                 <origin xyz="0 0 0" rpy="0 0 0" />
                 <geometry>
-                  <mesh filename="package://talos_description/meshes/gripper/fingertip_collision.STL" scale="1 1 1"/>
+                  <mesh filename="package://talos_data/meshes/gripper/fingertip_collision.STL" scale="1 1 1"/>
                 </geometry>
               </collision>

File: urdf/head/head.urdf.xacro (robot description, xacro)
@@ -9,7 +9,7 @@
 <robot xmlns:xacro="http://ros.org/wiki/xacro">
   <!--File includes-->
-  <xacro:include filename="$(find talos_description)/urdf/deg_to_rad.xacro" />
-  <xacro:include filename="$(find talos_description)/urdf/head/head.transmission.xacro" />
-  <xacro:include filename="$(find talos_description)/urdf/sensors/orbbec_astra_pro.urdf.xacro" />
+  <xacro:include filename="$(find talos_data)/urdf/deg_to_rad.xacro" />
+  <xacro:include filename="$(find talos_data)/urdf/head/head.transmission.xacro" />
+  <xacro:include filename="$(find talos_data)/urdf/sensors/orbbec_astra_pro.urdf.xacro" />
   <xacro:include filename="$(find talos_description_calibration)/urdf/calibration/calibration_constants.urdf.xacro" />
   <!--Constant parameters-->
@@ -27,5 +27,5 @@
         <origin xyz="0 0 0" rpy="0 0 0" />
         <geometry>
-          <mesh filename="package://talos_description/meshes/head/head_1.stl" scale="1 1 1"/>
+          <mesh filename="package://talos_data/meshes/head/head_1.stl" scale="1 1 1"/>
         </geometry>
         <material name="DarkGrey" />
@@ -34,5 +34,5 @@
         <origin xyz="0 0 0" rpy="0 0 0" />
         <geometry>
-          <mesh filename="package://talos_description/meshes/head/head_1_collision.stl" scale="1 1 1"/>
+          <mesh filename="package://talos_data/meshes/head/head_1_collision.stl" scale="1 1 1"/>
         </geometry>
       </collision>
@@ -71,5 +71,5 @@
         <origin xyz="0 0 0" rpy="0 0 0" />
         <geometry>
-          <mesh filename="package://talos_description/meshes/head/head_2.stl" scale="1 1 1"/>
+          <mesh filename="package://talos_data/meshes/head/head_2.stl" scale="1 1 1"/>
         </geometry>
         <material name="LightGrey" />
@@ -78,5 +78,5 @@
         <origin xyz="0 0 0" rpy="0 0 0" />
         <geometry>
-          <mesh filename="package://talos_description/meshes/head/head_2_collision.stl" scale="1 1 1"/>
+          <mesh filename="package://talos_data/meshes/head/head_2_collision.stl" scale="1 1 1"/>
         </geometry>
       </collision>

File: urdf/leg/foot_collision_default.urdf.xacro (robot description, xacro)
@@ -5,5 +5,5 @@
             <origin xyz="0 0 0" rpy="0 0 0" />
             <geometry>
-                <mesh filename="package://talos_description/meshes/v2/ankle_X_collision.stl" scale="1 ${reflect*1} 1"/>
+                <mesh filename="package://talos_data/meshes/v2/ankle_X_collision.stl" scale="1 ${reflect*1} 1"/>
             </geometry>
         </collision>

File: urdf/leg/leg_passive.urdf.xacro (robot description, xacro)
@@ -35,4 +35,44 @@
       <dynamics friction="${leg_friction}" damping="${leg_damping}"/>
     </joint>
+    <link name="leg_${prefix}_1_link_passive">
+      <inertial>
+        <mass value="0.001"/>
+        <inertia ixx="0.001" ixy="0.0" ixz="0.0" iyy="0.001" iyz="0.0" izz="0.001" />
+        <origin rpy="0 0 0" xyz="0.0 0.0 0.0"/>
+      </inertial>
+    </link>
+    <joint name="leg_${prefix}_1_joint_passive" type="revolute">
+      <parent link="leg_${prefix}_1_link"/>
+      <child link="leg_${prefix}_1_link_passive"/>
+      <origin xyz="0.0 0.0 0.0"
+              rpy="0.00000 0.00000 0.00000"/>
+      <axis xyz="0 1 0" />
+      <limit lower="${(-180.0)*deg_to_rad}" upper="${(180.0)*deg_to_rad}" effort="100" velocity="3.87" />
+      <dynamics friction="970.0" damping="0.0"/>
+    </joint>
+    <gazebo>
+      <plugin filename="libSpringPlugin.so" name="spring_leg_${prefix}_1_joint_passive">
+        <joint_spring>leg_${prefix}_1_joint_passive</joint_spring>
+        <kp>970.0</kp>
+        <kd>0.0</kd>
+      </plugin>
+    </gazebo>
+    <!-- Joint hip_x (mesh link) : child link hip_y -> parent link hip_z -->
+    <!-- <link name="leg_${prefix}_2_link_passive"> -->
+    <!--   <inertial> -->
+    <!--     <mass value="0.001"/> -->
+    <!--     <inertia ixx="0.001" ixy="0.0" ixz="0.0" iyy="0.001" iyz="0.0" izz="0.001" /> -->
+    <!--     <origin rpy="0 0 0" xyz="0.0 0.0 0.0"/> -->
+    <!--   </inertial> -->
+    <!-- </link> -->
+    <!-- <joint name="leg_${prefix}_2_joint_passive" type="revolute"> -->
+    <!--   <parent link="leg_${prefix}_1_link_passive"/> -->
+    <!--   <child link="leg_${prefix}_2_link_passive"/> -->
+    <!--   <origin xyz="0.0 0.0 0.0" -->
+    <!--           rpy="0.00000 0.00000 0.00000"/> -->
+    <!--   <axis xyz="0 1 0" /> -->
+    <!--   <limit lower="${(-180.0)*deg_to_rad}" upper="${(180.0)*deg_to_rad}" effort="100" velocity="3.87" /> -->
+    <!--   <dynamics friction="970.0" damping="0.0"/> -->
+    <!-- </joint> -->
     <!-- Joint hip_x (mesh link) : child link hip_y -> parent link hip_z -->
     <link name="leg_${prefix}_2_link">
@@ -53,5 +93,5 @@
     </link>
     <joint name="leg_${prefix}_2_joint" type="revolute">
-      <parent link="leg_${prefix}_1_link"/>
+      <parent link="leg_${prefix}_1_link_passive"/>
       <child link="leg_${prefix}_2_link"/>
       <origin xyz="0.00000 0.00000 0.00000"

File: urdf/sensors/orbbec_astra_pro.urdf.xacro (robot description, xacro)
@@ -18,5 +18,5 @@
 -->
 <robot xmlns:xacro="http://ros.org/wiki/xacro">
-  <xacro:include filename="$(find talos_description)/urdf/sensors/orbbec_astra_pro.gazebo.xacro" />
+  <xacro:include filename="$(find talos_data)/urdf/sensors/orbbec_astra_pro.gazebo.xacro" />
   <!-- Macro -->
   <xacro:macro name="orbbec_astra_pro" params="name parent *origin *optical_origin">
@@ -35,5 +35,5 @@
         <origin xyz="0 0 0" rpy="0 0 0"/>
         <geometry>
-          <mesh filename="package://talos_description/meshes/sensors/orbbec/orbbec.STL" />
+          <mesh filename="package://talos_data/meshes/sensors/orbbec/orbbec.STL" />
         </geometry>
         <material name="DarkGrey">

File: urdf/talos_full_common.urdf.xacro (robot description, xacro)
@@ -16,7 +16,13 @@
   <xacro:include filename="$(find talos_data)/urdf/torso/torso.urdf.xacro" />
   <xacro:include filename="$(find talos_data)/urdf/head/head.urdf.xacro" />
-  <xacro:include filename="$(find talos_data)/urdf/arm/arm_v2.urdf.xacro" />
+  <xacro:include filename="$(find talos_data)/urdf/arm/arm.urdf.xacro" />
   <xacro:include filename="$(find talos_data)/urdf/sensors/ftsensor.urdf.xacro" />
-  <xacro:include filename="$(find talos_data)/urdf/leg/leg.urdf.xacro" />
+  <xacro:include filename="$(find talos_data)/urdf/gripper/gripper.urdf.xacro" />
+  <!--  <xacro:if value="$(arg enable_leg_passive)"> -->
+    <xacro:include filename="$(find talos_data)/urdf/leg/leg_passive.urdf.xacro" />
+  <!-- </xacro:if> -->
+  <!-- <xacro:unless value="$(arg enable_leg_passive)">
+    <xacro:include filename="$(find talos_data)/urdf/leg/leg.urdf.xacro" />
+  </xacro:unless> -->
   <xacro:include filename="$(find talos_data)/urdf/leg/foot_collision_$(arg foot_collision).urdf.xacro" />
   <xacro:include filename="$(find talos_description_inertial)/urdf/inertial.xacro" />
@@ -26,8 +32,10 @@
   </xacro:if>
   <xacro:talos_head name="head" parent="torso_2_link"/>
-  <xacro:talos_arm name="arm" parent="torso_2_link" side="left" reflect="1"/>
-  <xacro:talos_arm name="arm" parent="torso_2_link" side="right" reflect="-1"/>
+  <xacro:talos_arm name="arm" parent="torso_2_link" side="left" reflect="1" />
+  <xacro:talos_arm name="arm" parent="torso_2_link" side="right" reflect="-1" />
   <xacro:ft_sensor name="wrist" parent="arm_right_7_link" side="right" reflect="1"  />
   <xacro:ft_sensor name="wrist" parent="arm_left_7_link"  side="left"  reflect="-1" />
+  <xacro:talos_gripper name="gripper_left" parent="wrist_left_ft_tool_link" reflect="1" />
+  <xacro:talos_gripper name="gripper_right" parent="wrist_right_ft_tool_link" reflect="-1" />
   <xacro:talos_leg prefix="left"  reflect="1" />
   <xacro:talos_leg prefix="right" reflect="-1" />

File: urdf/torso/torso.urdf.xacro (robot description, xacro)
@@ -9,7 +9,7 @@
 <robot xmlns:xacro="http://ros.org/wiki/xacro">
   <!--File includes-->
-  <xacro:include filename="$(find talos_description)/urdf/deg_to_rad.xacro" />
-  <xacro:include filename="$(find talos_description)/urdf/torso/torso.transmission.xacro" />
-  <xacro:include filename="$(find talos_description)/urdf/sensors/imu.urdf.xacro" />
+  <xacro:include filename="$(find talos_data)/urdf/deg_to_rad.xacro" />
+  <xacro:include filename="$(find talos_data)/urdf/torso/torso.transmission.xacro" />
+  <xacro:include filename="$(find talos_data)/urdf/sensors/imu.urdf.xacro" />
  <!--Constant parameters-->
   <xacro:property name="torso_max_vel"  value="5.4" />
@@ -25,5 +25,5 @@
         <origin xyz="0 0 0" rpy="0 0 0" />
         <geometry>
-          <mesh filename="package://talos_description/meshes/torso/torso_2.STL" scale="1 1 1"/>
+          <mesh filename="package://talos_data/meshes/torso/torso_2.STL" scale="1 1 1"/>
         </geometry>
         <material name="LightGrey" />
@@ -32,5 +32,5 @@
         <origin xyz="0 0 0" rpy="0 0 0" />
         <geometry>
-          <mesh filename="package://talos_description/meshes/torso/torso_2_collision.STL" scale="1 1 1"/>
+          <mesh filename="package://talos_data/meshes/torso/torso_2_collision.STL" scale="1 1 1"/>
         </geometry>
       </collision>
@@ -44,5 +44,5 @@
         <origin xyz="0 0 0" rpy="0 0 0" />
         <geometry>
-          <mesh filename="package://talos_description/meshes/torso/torso_1.STL" scale="1 1 1"/>
+          <mesh filename="package://talos_data/meshes/torso/torso_1.STL" scale="1 1 1"/>
         </geometry>
         <material name="LightGrey" />
@@ -51,5 +51,5 @@
         <origin xyz="0 0 0" rpy="0 0 0" />
         <geometry>
-          <mesh filename="package://talos_description/meshes/torso/torso_1.STL" scale="1 1 1"/>
+          <mesh filename="package://talos_data/meshes/torso/torso_1.STL" scale="1 1 1"/>
         </geometry>
       </collision>
@@ -78,5 +78,5 @@
         <origin xyz="0 0 0" rpy="0 0 0" />
         <geometry>
-          <mesh filename="package://talos_description/meshes/torso/base_link.STL" scale="1 1 1"/>
+          <mesh filename="package://talos_data/meshes/torso/base_link.STL" scale="1 1 1"/>
         </geometry>
         <material name="LightGrey" />
@@ -85,5 +85,5 @@
         <origin xyz="0 0 0" rpy="0 0 0" />
         <geometry>
-          <mesh filename="package://talos_description/meshes/torso/base_link_collision.STL" scale="1 1 1"/>
+          <mesh filename="package://talos_data/meshes/torso/base_link_collision.STL" scale="1 1 1"/>
         </geometry>
       </collision>
