Commit message: Use full models of gripper inner bodies for collision checking

File: urdf/talos_full.urdf (robot description, URDF)
Before this commit: robot talos, 60 links, 59 joints
Links:
- link gripper_left_inner_double_link: geometry collision mesh filename=package://talos-data/meshes/gripper/inner_double.STL scale=1 1 1; visual mesh filename=package://talos-data/meshes/gripper/inner_double.STL scale=1 1 1
- link gripper_left_inner_single_link: geometry collision mesh filename=package://talos-data/meshes/gripper/inner_single.STL scale=1 1 1; visual mesh filename=package://talos-data/meshes/gripper/inner_single.STL scale=1 1 1
- link gripper_right_inner_double_link: geometry collision mesh filename=package://talos-data/meshes/gripper/inner_double.STL scale=1 1 1; visual mesh filename=package://talos-data/meshes/gripper/inner_double.STL scale=1 1 1
- link gripper_right_inner_single_link: geometry collision mesh filename=package://talos-data/meshes/gripper/inner_single.STL scale=1 1 1; visual mesh filename=package://talos-data/meshes/gripper/inner_single.STL scale=1 1 1

Commit message: [cmake] Remove srdf file + URDF fixes

File: urdf/talos_full.urdf (robot description, URDF)
Before this commit: robot talos, 60 links, 59 joints
Links:
- link leg_left_1_link: geometry collision mesh filename=package://talos_data/meshes/v2/hip_z_collision.stl scale=1 1 1; visual mesh filename=package://talos_data/meshes/v2/hip_z_lo_res.stl scale=1 1 1
- link leg_left_2_link: geometry collision mesh filename=package://talos_data/meshes/v2/hip_x_collision.stl scale=1 1 1; visual mesh filename=package://talos_data/meshes/v2/hip_x_lo_res.stl scale=1 1 1
- link leg_left_3_link: geometry collision mesh filename=package://talos_data/meshes/v2/hip_y_collision.stl scale=1 1 1; visual mesh filename=package://talos_data/meshes/v2/hip_y_lo_res.stl scale=1 1 1
- link leg_left_4_link: geometry collision mesh filename=package://talos_data/meshes/v2/knee_collision.stl scale=1 1 1; visual mesh filename=package://talos_data/meshes/v2/knee_lo_res.stl scale=1 1 1
- link leg_left_5_link: geometry collision mesh filename=package://talos_data/meshes/v2/ankle_Y_collision.stl scale=1 1 1; visual mesh filename=package://talos_data/meshes/v2/ankle_Y_lo_res.stl scale=1 1 1
- link leg_left_6_link: geometry collision box size=0.21 0.13 0.02; visual mesh filename=package://talos_data/meshes/v2/ankle_X_lo_res.stl scale=1 1 1
- link leg_right_1_link: geometry collision mesh filename=package://talos_data/meshes/v2/hip_z_collision.stl scale=1 -1 1; visual mesh filename=package://talos_data/meshes/v2/hip_z_lo_res.stl scale=1 -1 1
- link leg_right_2_link: geometry collision mesh filename=package://talos_data/meshes/v2/hip_x_collision.stl scale=1 -1 1; visual mesh filename=package://talos_data/meshes/v2/hip_x_lo_res.stl scale=1 -1 1
- link leg_right_3_link: geometry collision mesh filename=package://talos_data/meshes/v2/hip_y_collision.stl scale=1 -1 1; visual mesh filename=package://talos_data/meshes/v2/hip_y_lo_res.stl scale=1 -1 1
- link leg_right_4_link: geometry collision mesh filename=package://talos_data/meshes/v2/knee_collision.stl scale=1 -1 1; visual mesh filename=package://talos_data/meshes/v2/knee_lo_res.stl scale=1 -1 1
- link leg_right_5_link: geometry collision mesh filename=package://talos_data/meshes/v2/ankle_Y_collision.stl scale=1 -1 1; visual mesh filename=package://talos_data/meshes/v2/ankle_Y_lo_res.stl scale=1 -1 1
- link leg_right_6_link: geometry collision box size=0.21 0.13 0.02; visual mesh filename=package://talos_data/meshes/v2/ankle_X_lo_res.stl scale=1 -1 1

File: urdf/talos_full_v2.urdf (robot description, URDF)
Before this commit: robot talos, 60 links, 59 joints
Links:
- link arm_left_1_link: geometry collision mesh filename=package://talos_data/meshes/arm/arm_1_collision.STL scale=1 1 1; visual mesh filename=package://talos_data/meshes/arm/arm_1.STL scale=1 1 1
- link arm_left_2_link: geometry collision mesh filename=package://talos_data/meshes/arm/arm_2_collision.STL scale=1 1 1; visual mesh filename=package://talos_data/meshes/arm/arm_2.STL scale=1 1 1
- link arm_left_3_link: geometry collision mesh filename=package://talos_data/meshes/arm/arm_3_collision.STL scale=1 1 1; visual mesh filename=package://talos_data/meshes/arm/arm_3.STL scale=1 1 1
- link arm_left_4_link: geometry collision mesh filename=package://talos_data/meshes/arm/arm_4_collision.STL scale=1 1 1; visual mesh filename=package://talos_data/meshes/arm/arm_4.STL scale=1 1 1
- link arm_left_5_link: geometry collision mesh filename=package://talos_data/meshes/arm/arm_5_collision.STL scale=1 1 1; visual mesh filename=package://talos_data/meshes/arm/arm_5.STL scale=1 1 1
- link arm_left_6_link: geometry collision mesh filename=package://talos_data/meshes/arm/arm_6_collision.STL scale=1 1 1; visual mesh filename=package://talos_data/meshes/arm/arm_6.STL scale=1 1 1
- link arm_left_7_link: geometry collision mesh filename=package://talos_data/meshes/arm/arm_7_collision.STL scale=1 1 1; visual mesh filename=package://talos_data/meshes/arm/arm_7.STL scale=1 1 1
- link arm_right_1_link: geometry collision mesh filename=package://talos_data/meshes/arm/arm_1_collision.STL scale=1 -1 1; visual mesh filename=package://talos_data/meshes/arm/arm_1.STL scale=1 -1 1
- link arm_right_2_link: geometry collision mesh filename=package://talos_data/meshes/arm/arm_2_collision.STL scale=1 -1 1; visual mesh filename=package://talos_data/meshes/arm/arm_2.STL scale=1 -1 1
- link arm_right_3_link: geometry collision mesh filename=package://talos_data/meshes/arm/arm_3_collision.STL scale=1 -1 1; visual mesh filename=package://talos_data/meshes/arm/arm_3.STL scale=1 -1 1
- link arm_right_4_link: geometry collision mesh filename=package://talos_data/meshes/arm/arm_4_collision.STL scale=1 -1 1; visual mesh filename=package://talos_data/meshes/arm/arm_4.STL scale=1 -1 1
- link arm_right_5_link: geometry collision mesh filename=package://talos_data/meshes/arm/arm_5_collision.STL scale=1 -1 1; visual mesh filename=package://talos_data/meshes/arm/arm_5.STL scale=1 -1 1
- link arm_right_6_link: geometry collision mesh filename=package://talos_data/meshes/arm/arm_6_collision.STL scale=1 -1 1; visual mesh filename=package://talos_data/meshes/arm/arm_6.STL scale=1 -1 1
- link arm_right_7_link: geometry collision mesh filename=package://talos_data/meshes/arm/arm_7_collision.STL scale=1 -1 1; visual mesh filename=package://talos_data/meshes/arm/arm_7.STL scale=1 -1 1
- link base_link: geometry collision mesh filename=package://talos_data/meshes/torso/base_link_collision.STL scale=1 1 1; visual mesh filename=package://talos_data/meshes/torso/base_link.STL scale=1 1 1
- link gripper_left_base_link: geometry collision mesh filename=package://talos_data/meshes/gripper/base_link_collision.STL scale=1 1 1; visual mesh filename=package://talos_data/meshes/gripper/base_link.STL scale=1 1 1
- link gripper_left_fingertip_1_link: geometry collision mesh filename=package://talos_data/meshes/gripper/fingertip_collision.STL scale=1 1 1; visual mesh filename=package://talos_data/meshes/gripper/fingertip.STL scale=1 1 1
- link gripper_left_fingertip_2_link: geometry collision mesh filename=package://talos_data/meshes/gripper/fingertip_collision.STL scale=1 1 1; visual mesh filename=package://talos_data/meshes/gripper/fingertip.STL scale=1 1 1
- link gripper_left_fingertip_3_link: geometry collision mesh filename=package://talos_data/meshes/gripper/fingertip_collision.STL scale=1 1 1; visual mesh filename=package://talos_data/meshes/gripper/fingertip.STL scale=1 1 1
- link gripper_left_inner_double_link: geometry collision mesh filename=package://talos_data/meshes/gripper/inner_double_collision.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 scale=1 1 1; visual mesh filename=package://talos_data/meshes/gripper/inner_double.STL scale=1 1 1
- link gripper_left_inner_single_link: geometry collision mesh filename=package://talos_data/meshes/gripper/inner_single_collision.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 scale=1 1 1; visual mesh filename=package://talos_data/meshes/gripper/inner_single.STL scale=1 1 1
- link gripper_left_motor_double_link: geometry collision mesh filename=package://talos_data/meshes/gripper/gripper_motor_double_co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 scale=1 1 1; visual mesh filename=package://talos_data/meshes/gripper/gripper_motor_double.STL scale=1 1 1
- link gripper_left_motor_single_link: geometry collision mesh filename=package://talos_data/meshes/gripper/gripper_motor_single_co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 scale=1 1 1; visual mesh filename=package://talos_data/meshes/gripper/gripper_motor_single.STL scale=1 1 1
- link gripper_right_base_link: geometry collision mesh filename=package://talos_data/meshes/gripper/base_link_collision.STL scale=1 1 1; visual mesh filename=package://talos_data/meshes/gripper/base_link.STL scale=1 1 1
- link gripper_right_fingertip_1_link: geometry collision mesh filename=package://talos_data/meshes/gripper/fingertip_collision.STL scale=1 1 1; visual mesh filename=package://talos_data/meshes/gripper/fingertip.STL scale=1 1 1
- link gripper_right_fingertip_2_link: geometry collision mesh filename=package://talos_data/meshes/gripper/fingertip_collision.STL scale=1 1 1; visual mesh filename=package://talos_data/meshes/gripper/fingertip.STL scale=1 1 1
- link gripper_right_fingertip_3_link: geometry collision mesh filename=package://talos_data/meshes/gripper/fingertip_collision.STL scale=1 1 1; visual mesh filename=package://talos_data/meshes/gripper/fingertip.STL scale=1 1 1
- link gripper_right_inner_double_link: geometry collision mesh filename=package://talos_data/meshes/gripper/inner_double_collision.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 scale=1 1 1; visual mesh filename=package://talos_data/meshes/gripper/inner_double.STL scale=1 1 1
- link gripper_right_inner_single_link: geometry collision mesh filename=package://talos_data/meshes/gripper/inner_single_collision.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 scale=1 1 1; visual mesh filename=package://talos_data/meshes/gripper/inner_single.STL scale=1 1 1
- link gripper_right_motor_double_link: geometry collision mesh filename=package://talos_data/meshes/gripper/gripper_motor_double_co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 scale=1 1 1; visual mesh filename=package://talos_data/meshes/gripper/gripper_motor_double.STL scale=1 1 1
- link gripper_right_motor_single_link: geometry collision mesh filename=package://talos_data/meshes/gripper/gripper_motor_single_co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 scale=1 1 1; visual mesh filename=package://talos_data/meshes/gripper/gripper_motor_single.STL scale=1 1 1
- link head_1_link: geometry collision mesh filename=package://talos_data/meshes/head/head_1_collision.stl scale=1 1 1; visual mesh filename=package://talos_data/meshes/head/head_1.stl scale=1 1 1
- link head_2_link: geometry collision mesh filename=package://talos_data/meshes/head/head_2_collision.stl scale=1 1 1; visual mesh filename=package://talos_data/meshes/head/head_2.stl scale=1 1 1
- link leg_left_1_link: geometry collision mesh filename=package://talos_data/meshes/v2/hip_z_collision.stl scale=1 1 1; visual mesh filename=package://talos_data/meshes/v2/hip_z_lo_res.stl scale=1 1 1
- link leg_left_2_link: geometry collision mesh filename=package://talos_data/meshes/v2/hip_x_collision.stl scale=1 1 1; visual mesh filename=package://talos_data/meshes/v2/hip_x_lo_res.stl scale=1 1 1
- link leg_left_3_link: geometry collision mesh filename=package://talos_data/meshes/v2/hip_y_collision.stl scale=1 1 1; visual mesh filename=package://talos_data/meshes/v2/hip_y_lo_res.stl scale=1 1 1
- link leg_left_4_link: geometry collision mesh filename=package://talos_data/meshes/v2/knee_collision.stl scale=1 1 1; visual mesh filename=package://talos_data/meshes/v2/knee_lo_res.stl scale=1 1 1
- link leg_left_5_link: geometry collision mesh filename=package://talos_data/meshes/v2/ankle_Y_collision.stl scale=1 1 1; visual mesh filename=package://talos_data/meshes/v2/ankle_Y_lo_res.stl scale=1 1 1
- link leg_left_6_link: geometry collision box size=0.21 0.13 0.02; visual mesh filename=package://talos_data/meshes/v2/ankle_X_lo_res.stl scale=1 1 1
- link leg_right_1_link: geometry collision mesh filename=package://talos_data/meshes/v2/hip_z_collision.stl scale=1 -1 1; visual mesh filename=package://talos_data/meshes/v2/hip_z_lo_res.stl scale=1 -1 1
- link leg_right_2_link: geometry collision mesh filename=package://talos_data/meshes/v2/hip_x_collision.stl scale=1 -1 1; visual mesh filename=package://talos_data/meshes/v2/hip_x_lo_res.stl scale=1 -1 1
- link leg_right_3_link: geometry collision mesh filename=package://talos_data/meshes/v2/hip_y_collision.stl scale=1 -1 1; visual mesh filename=package://talos_data/meshes/v2/hip_y_lo_res.stl scale=1 -1 1
- link leg_right_4_link: geometry collision mesh filename=package://talos_data/meshes/v2/knee_collision.stl scale=1 -1 1; visual mesh filename=package://talos_data/meshes/v2/knee_lo_res.stl scale=1 -1 1
- link leg_right_5_link: geometry collision mesh filename=package://talos_data/meshes/v2/ankle_Y_collision.stl scale=1 -1 1; visual mesh filename=package://talos_data/meshes/v2/ankle_Y_lo_res.stl scale=1 -1 1
- link leg_right_6_link: geometry collision box size=0.21 0.13 0.02; visual mesh filename=package://talos_data/meshes/v2/ankle_X_lo_res.stl scale=1 -1 1
- link rgbd_link: geometry collision box size=0.04 0.185 0.03; visual mesh filename=package://talos_data/meshes/sensors/orbbec/orbbec.STL
- link torso_1_link: geometry collision mesh filename=package://talos_data/meshes/torso/torso_1.STL scale=1 1 1; visual mesh filename=package://talos_data/meshes/torso/torso_1.STL scale=1 1 1
- link torso_2_link: geometry collision mesh filename=package://talos_data/meshes/torso/torso_2_collision.STL scale=1 1 1; visual mesh filename=package://talos_data/meshes/torso/torso_2.STL scale=1 1 1
