Commit message: Fix talos_reduced_v2.urdf
* Make fixed the following joints:
* gripper_left_inner_double_joint
* gripper_left_inner_single_joint
* gripper_left_motor_single_joint
* gripper_right_inner_double_joint
* gripper_right_inner_single_joint
* gripper_right_motor_single_joint

File: urdf/talos_reduced_v2.urdf (robot description, URDF)
Before this commit: robot talos, 60 links, 59 joints
Joints:
- joint gripper_left_inner_double_joint: type revolute -> fixed
- joint gripper_left_inner_single_joint: type revolute -> fixed
- joint gripper_left_motor_single_joint: type revolute -> fixed
- joint gripper_right_inner_double_joint: type revolute -> fixed
- joint gripper_right_inner_single_joint: type revolute -> fixed
- joint gripper_right_motor_single_joint: type revolute -> fixed
