Commit message: [urdf] change collision geometry for ankle : use convex mesh instead of box

File: urdf/talos_reduced.urdf (robot description, URDF)
Before this commit: robot talos, 60 links, 59 joints
Links:
- link leg_left_6_link: geometry collision mesh filename=package://talos_data/meshes/v2/ankle_X_collision.stl scale=1 1 1; visual mesh filename=package://talos_data/meshes/v2/ankle_X_lo_res.stl scale=1 1.0 1
- link leg_right_6_link: geometry collision mesh filename=package://talos_data/meshes/v2/ankle_X_collision.stl scale=1 -1 1; visual mesh filename=package://talos_data/meshes/v2/ankle_X_lo_res.stl scale=1 -1.0 1
