Commit message: Add fixed link.

File: urdf/talos_full_common.urdf.xacro (robot description, xacro)
@@ -19,8 +19,9 @@
   <xacro:include filename="$(find talos_data)/urdf/sensors/ftsensor.urdf.xacro" />
   <xacro:include filename="$(find talos_data)/urdf/gripper/gripper.urdf.xacro" />
-  <!--  <xacro:if value="$(arg enable_leg_passive)"> -->
+  <xacro:if value="$(arg enable_leg_passive)">
     <xacro:include filename="$(find talos_data)/urdf/leg/leg_passive.urdf.xacro" />
-  <!-- </xacro:if> -->
-  <!-- <xacro:unless value="$(arg enable_leg_passive)">
+  </xacro:if>
+  <xacro:unless name="var_enable_leg_passive" value="$(arg enable_leg_passive)"/>
+  <xacro:unless value="${var_enable_leg_passive != 'true'}">
     <xacro:include filename="$(find talos_data)/urdf/leg/leg.urdf.xacro" />
   </xacro:unless> -->

File: urdf/torso/torso.urdf.xacro (robot description, xacro)
@@ -89,4 +89,11 @@
       </collision>
     </link>
+    <!-- <xacro:if value="$(arg enable_fixed_robot)"> -->
+      <link name="world"/>
+      <joint name="fixed" type="fixed">
+        <parent link="world"/>
+        <child link="base_link"/>
+      </joint>
+    <!-- </xacro:if> -->
     <joint name="${name}_2_joint" type="revolute">
       <parent link="${name}_1_link"/>
