Commit message: Remove dependency to realsense2_description
  Replace camera models by boxes.

File: urdf/talos_full_v2_with_lidar.urdf (robot description, URDF)
Before this commit: robot talos, 75 links, 74 joints
Links:
- link head_d435_camera_link: geometry collision box size=0.02505 0.09 0.025; visual box size=0.090 0.025 0.02505
- link head_t265_camera_link: geometry collision box size=0.090 0.025 0.02505; visual box size=0.090 0.025 0.02505
