Commit message: Fix SpringPlugin + add transmission to leg_{prefix}_1_joint_passive

File: urdf/leg/leg_passive.urdf.xacro (robot description, xacro)
@@ -58,4 +58,14 @@
       </plugin>
     </gazebo>
+    <transmission name="leg_${prefix}_1_passive_trans">
+      <type>transmission_interface/SimpleTransmission</type>
+      <actuator name="leg_${prefix}_1_motor" >
+        <mechanicalReduction>${reduction}</mechanicalReduction>
+      </actuator>
+      <joint name="leg_${prefix}_1_joint">
+        <hardwareInterface>hardware_interface/PositionJointInterface</hardwareInterface>
+        <hardwareInterface>hardware_interface/EffortJointInterface</hardwareInterface>
+      </joint>
+    </transmission>
     <!-- Joint hip_x (mesh link) : child link hip_y -> parent link hip_z -->
     <!-- <link name="leg_${prefix}_2_link_passive"> -->

Commit message: Fix passive tranmission to have the passive joints in the state of the robot.

File: urdf/leg/leg_passive.urdf.xacro (robot description, xacro)
@@ -61,7 +61,7 @@
       <type>transmission_interface/SimpleTransmission</type>
       <actuator name="leg_${prefix}_1_motor" >
-        <mechanicalReduction>${reduction}</mechanicalReduction>
+        <mechanicalReduction>1.0</mechanicalReduction>
       </actuator>
-      <joint name="leg_${prefix}_1_joint">
+      <joint name="leg_${prefix}_1_joint_passive">
         <hardwareInterface>hardware_interface/PositionJointInterface</hardwareInterface>
         <hardwareInterface>hardware_interface/EffortJointInterface</hardwareInterface>

Commit message: [urdf] Changing the spring axis from Y to X.

File: urdf/leg/leg_passive.urdf.xacro (robot description, xacro)
@@ -47,5 +47,5 @@
       <origin xyz="0.0 0.0 0.0"
               rpy="0.00000 0.00000 0.00000"/>
-      <axis xyz="0 1 0" />
+      <axis xyz="1 0 0" />
       <limit lower="${(-180.0)*deg_to_rad}" upper="${(180.0)*deg_to_rad}" effort="100" velocity="3.87" />
       <dynamics friction="970.0" damping="0.0"/>
